File: A52GL/1_Top/A52GL_Top.kicad_pcb (KiCad board)
At the start: 2 copper layers, 315.8 x 99.2 mm, 89 parts, among them J10 Conn_01x01, J11 Conn_01x01, J12 Conn_01x01, J13 Conn_01x01, J14 Conn_01x01, J15 Conn_01x01, J16 Conn_01x01, J17 Conn_01x01, J2 Conn_01x01, J3 Conn_01x01, J4 Conn_01x01, J5 Conn_01x01, J6 Conn_01x01, J7 Conn_01x01, J8 Conn_01x01, J9 Conn_01x01, SW1 SW_PUSH, SW2 KEY_SWITCH, SW3 SW_PUSH, SW4 KEY_SWITCH, SW4 SW_PUSH, SW5 SW_PUSH, SW7 SW_PUSH, SW8 SW_PUSH

Commit message: いっぱい追加
Parts:
- removed the SW4 at (292.9, 57.1)
- removed the SW4 at (271.5, 66.7)
- removed the SW4 at (233.4, 66.7)
- removed the SW4 at (238.1, 28.6)
- removed the SW4 at (214.3, 66.7)
- removed the SW4 at (161.9, 28.6)
- removed the SW4 at (176.2, 66.7)
- removed the SW4 at (181.0, 28.6)
- removed the SW4 at (200.0, 28.6)
- removed the SW4 at (195.3, 66.7)
- removed the SW4 at (142.9, 28.6)
- removed the SW4 at (40.5, 85.7)
- removed the SW4 at (138.1, 66.7)
- removed the SW4 at (123.8, 28.6)
- removed the SW4 at (157.2, 66.7)
- removed the SW4 at (119.1, 66.7)
- removed the SW4 at (104.8, 28.6)
- removed the SW4 at (100.0, 66.7)
- removed the SW4 at (85.7, 28.6)
- removed the SW4 at (81.0, 66.7)
- removed the SW4 at (66.7, 28.6)
- removed the SW4 at (61.9, 66.7)
- removed the SW4 at (276.2, 28.6)
- removed the SW4 at (295.3, 28.6)
- removed the SW4 at (314.3, 66.7)
- removed the SW4 at (314.3, 28.6)
- removed the SW4 at (252.4, 66.7)
- removed the SW4 at (219.1, 28.6)
- removed the SW4 at (257.2, 28.6)
- removed the SW5 at (221.5, 104.8)
- removed the SW5 at (245.3, 104.8)
- removed the SW5 at (178.6, 104.8)
- removed the SW8 at (269.1, 85.7)
- removed the SW8 at (266.7, 47.6)
- removed the SW8 at (247.7, 47.6)
- removed the SW8 at (228.6, 47.6)
- removed the SW8 at (242.9, 85.7)
- removed the SW8 at (295.3, 85.7)
- removed the SW8 at (190.5, 47.6)
- removed the SW8 at (171.4, 47.6)
- removed the SW8 at (204.8, 85.7)
- removed the SW8 at (223.8, 85.7)
- removed the SW8 at (209.6, 47.6)
- removed the SW8 at (200.0, 104.8)
- removed the SW8 at (185.7, 85.7)
- removed the SW8 at (128.6, 85.7)
- removed the SW8 at (152.4, 47.6)
- removed the SW8 at (147.6, 85.7)
- removed the SW8 at (133.3, 47.6)
- removed the SW8 at (166.7, 85.7)
- removed the SW8 at (114.3, 47.6)
- removed the SW8 at (95.2, 104.8)
- removed the SW8 at (109.5, 85.7)
- removed the SW8 at (95.2, 47.6)
- removed the SW8 at (138.1, 104.8)
- removed the SW8 at (90.5, 85.7)
- removed the SW8 at (76.2, 47.6)
- removed the SW8 at (71.4, 85.7)
- removed the SW8 at (157.2, 104.8)
- removed the SW8 at (295.3, 104.8)
- removed the SW8 at (314.3, 104.8)
- removed the SW8 at (276.2, 104.8)
- removed the SW8 at (314.3, 47.6)
- removed the SW8 at (314.3, 85.7)
- added SW10: SW_PUSH, kbd_SW_Hole:SW_Hole, F.Cu at (76.0, 32.6)
- added SW12: SW_PUSH, kbd_SW_Hole:SW_Hole, F.Cu at (94.7, 36.0)
- added SW13: SW_PUSH, kbd_SW_Hole:SW_Hole, F.Cu at (96.1, 55.5)
- added SW14: SW_PUSH, kbd_SW_Hole:SW_Hole, F.Cu at (77.3, 52.2)
- added SW15: SW_PUSH, kbd_SW_Hole:SW_Hole, F.Cu at (82.5, 72.5)
- added SW16: SW_PUSH, kbd_SW_Hole:SW_Hole, F.Cu at (79.2, 91.3)
- added SW16: SW_PUSH, kbd_SW_Hole:SW_Hole, F.Cu at (120.0, 79.1)
- added SW18: SW_PUSH, kbd_SW_Hole:SW_Hole, F.Cu at (132.2, 42.6)
- added SW19: SW_PUSH, kbd_SW_Hole:SW_Hole, F.Cu at (133.6, 62.2)
- added SW20: SW_PUSH, kbd_SW_Hole:SW_Hole, F.Cu at (101.3, 75.8)
- added SW20: SW_PUSH, kbd_SW_Hole:SW_Hole, F.Cu at (138.8, 82.4)
- added SW21: SW_PUSH, kbd_SW_Hole:SW_Hole, F.Cu at (175.6, 62.2)
- added SW22: SW_PUSH, kbd_SW_Hole:SW_Hole, F.Cu at (170.8, 82.4)
- added SW23: SW_PUSH, kbd_SW_Hole:SW_Hole_2.25, F.Cu at (185.8, 99.1)
- added SW23: SW_PUSH, kbd_SW_Hole:SW_Hole, F.Cu at (113.5, 39.3)
- added SW24: SW_PUSH, kbd_SW_Hole:SW_Hole, F.Cu at (114.8, 58.9)
- added SW25: SW_PUSH, kbd_SW_Hole:SW_Hole, F.Cu at (186.3, 41.0)
- added SW27: SW_PUSH, kbd_SW_Hole:SW_Hole, F.Cu at (205.1, 37.7)
- added SW28: SW_PUSH, kbd_SW_Hole:SW_Hole, F.Cu at (213.1, 55.6)
- added SW29: SW_PUSH, kbd_SW_Hole:SW_Hole, F.Cu at (208.3, 75.8)
- added SW30: SW_PUSH, kbd_SW_Hole:SW_Hole, F.Cu at (135.5, 101.2)
- added SW32: SW_PUSH, kbd_SW_Hole:SW_Hole, F.Cu at (167.5, 44.3)
- added SW38: SW_PUSH, kbd_SW_Hole:SW_Hole, F.Cu at (194.3, 58.9)
- added SW39: SW_PUSH, kbd_SW_Hole:SW_Hole, F.Cu at (189.6, 79.1)
- added SW46: SW_PUSH, kbd_SW_Hole:SW_Hole, F.Cu at (223.8, 34.4)
- added SW47: SW_PUSH, kbd_SW_Hole:SW_Hole, F.Cu at (231.8, 52.3)
- added SW48: SW_PUSH, kbd_SW_Hole:SW_Hole, F.Cu at (227.1, 72.5)
- added SW49: SW_PUSH, kbd_SW_Hole:SW_Hole_1.25, F.Cu at (218.7, 93.3)
- added SW51: SW_PUSH, kbd_SW_Hole:SW_Hole, F.Cu at (244.3, 31.8)
- added SW51: SW_PUSH, kbd_SW_Hole:SW_Hole, F.Cu at (263.3, 32.6)
- added SW52: SW_PUSH, kbd_SW_Hole:SW_Hole, F.Cu at (252.4, 51.6)
- added SW53: SW_PUSH, kbd_SW_Hole:SW_Hole, F.Cu at (247.7, 89.7)
- added SW53: SW_PUSH, kbd_SW_Hole:SW_Hole, F.Cu at (247.7, 70.7)
- added SW53: SW_PUSH, kbd_SW_Hole:SW_Hole, F.Cu at (266.7, 70.7)
- added SW54: SW_PUSH, kbd_SW_Hole:SW_Hole, F.Cu at (271.5, 94.5)
- added SW56: SW_PUSH, kbd_SW_Hole:SW_Hole, F.Cu at (282.4, 32.6)
- added SW57: SW_PUSH, kbd_SW_Hole:SW_Hole, F.Cu at (271.5, 51.6)
- added SW58: SW_PUSH, kbd_SW_Hole:SW_Hole, F.Cu at (290.5, 75.4)
- added SW59: SW_PUSH, kbd_SW_Hole:SW_Hole, F.Cu at (290.5, 94.5)
- added SW61: SW_PUSH, kbd_SW_Hole:SW_Hole_1.5, F.Cu at (306.2, 32.6)
- added SW62: SW_PUSH, kbd_SW_Hole:SW_Hole_2.25, F.Cu at (302.4, 51.6)
- added SW63: SW_PUSH, kbd_SW_Hole:SW_Hole, F.Cu at (314.3, 70.7)
- added SW64: SW_PUSH, kbd_SW_Hole:SW_Hole, F.Cu at (309.6, 94.5)
- SW2: footprint kbd_SW_Hole:SW_Hole_1.5 -> kbd_SW_Hole:SW_Hole_2
- moved SW5 97.2 mm to (35.3, 51.6)
- moved SW2 88.5 mm to (107.3, 96.2), turned to 170 degrees
- moved SW7 53.3 mm to (56.8, 51.6)
- moved SW7 24.3 mm to (54.8, 89.7)
- moved SW8 23.5 mm to (61.9, 70.7)
- moved SW7 15.1 mm to (31.0, 89.7)
- moved SW4 8.73 mm to (55.4, 32.6)
- moved SW4 8.73 mm to (36.3, 32.6)
- moved SW6 4.00 mm to (35.7, 70.7)
- renumbered SW1 to SW4, SW3 to SW6
