File: J73GL/2_Assemble/J73GL_Assemble.kicad_pcb (KiCad board)
At the start: 2 copper layers, 305.2 x 99.2 mm, 223 parts, among them J1 Conn_01x02, SW1 SW_PUSH, SW10 SW_PUSH, SW11 SW_PUSH, SW12 SW_PUSH, SW13 SW_PUSH, SW14 SW_PUSH, SW15 SW_PUSH, SW16 SW_PUSH, SW17 SW_PUSH, SW18 SW_PUSH, SW19 SW_PUSH, SW2 KEY_SWITCH, SW2 SW_PUSH, SW20 SW_PUSH, SW21 SW_PUSH, SW22 SW_PUSH, SW23 SW_PUSH, SW24 SW_PUSH, SW25 SW_PUSH, SW26 SW_PUSH, SW27 SW_PUSH, SW28 SW_PUSH, SW29 SW_PUSH, SW3 SW_PUSH, SW30 SW_PUSH, SW31 SW_PUSH, SW32 SW_PUSH, SW33 SW_PUSH, SW34 SW_PUSH, SW35 SW_PUSH, SW36 SW_PUSH, SW37 SW_PUSH, SW38 SW_PUSH, SW39 SW_PUSH, SW4 SW_PUSH, SW40 SW_PUSH, SW41 SW_PUSH, SW42 SW_PUSH, SW43 SW_PUSH, SW44 SW_PUSH, SW45 SW_PUSH, SW46 SW_PUSH, SW47 SW_PUSH, SW48 SW_PUSH, SW49 SW_PUSH, SW5 SW_PUSH, SW50 SW_PUSH, SW51 SW_PUSH, SW52 SW_PUSH, SW53 SW_PUSH, SW54 SW_PUSH, SW55 SW_PUSH, SW56 SW_PUSH, SW57 SW_PUSH, SW58 SW_PUSH, SW59 SW_PUSH, SW6 SW_PUSH, SW60 SW_PUSH, SW61 SW_PUSH, SW62 SW_PUSH, SW63 SW_PUSH, SW64 SW_PUSH, SW65 SW_PUSH, SW66 SW_PUSH, SW67 SW_PUSH, SW68 SW_PUSH, SW69 SW_PUSH, SW7 SW_PUSH, SW70 SW_PUSH, SW71 SW_PUSH, SW72 SW_PUSH, SW73 SW_PUSH, SW74 SW_PUSH, SW8 SW_PUSH, SW9 SW_PUSH, U1 BLEMicroPro

Commit message: 色々更新
・J74GLからJ73GLに変更
・色々進捗
Parts:
- SW74, U1: moved to B.Cu
- moved SW74 69.2 mm to (266.7, 38.1), turned to 0 degrees
- moved L1 0.50 mm to (314.3, 24.3)
- moved L9 0.50 mm to (295.3, 24.3)
- moved U1 0.10 mm to (307.2, 28.9), turned to 270 degrees
- renumbered SW2 to SW75
Routing:
- net GND: track 0.00 -> 2215.3 mm, vias 0 -> 72
- net VCC: track 0.00 -> 2184.3 mm
- net Col0: track 0.00 -> 525.9 mm, vias 0 -> 12
- net Row4: track 0.00 -> 518.8 mm, vias 0 -> 2
- net Col1: track 0.00 -> 513.6 mm, vias 0 -> 14
- net Col5: track 0.00 -> 494.9 mm, vias 0 -> 15
- net Col2: track 0.00 -> 491.2 mm, vias 0 -> 12
- net Col3: track 0.00 -> 473.3 mm, vias 0 -> 13
- net Row2: track 0.00 -> 431.5 mm, vias 0 -> 10
- net Row1: track 0.00 -> 419.5 mm, vias 0 -> 5
- net Row0: track 0.00 -> 417.8 mm, vias 0 -> 6
- net Col6: track 0.00 -> 398.8 mm, vias 0 -> 12
- net Col4: track 0.00 -> 386.5 mm, vias 0 -> 12
- net Row3: track 0.00 -> 346.1 mm, vias 0 -> 5
- net Bat+: track 0.00 -> 121.2 mm
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
Commit message: いっぱい追加
Parts:
- D1, D10, D11, D12, D13, D14, D15, D16, D17, D18, D19, D2, D20, D21, D22, D23, D24, D25, D26, D27, D28, D29, D3, D30, D31, D32, D33, D34, D35, D36, D37, D38, D39, D4, D40, D41, D42, D43, D44, D45, D46, D47, D48, D49, D5, D50, D51, D52, D53, D54, D55, D56, D57, D58, D59, D6, D60, D61, D62, D63, D64, D65, D66, D67, D68, D69, D7, D70, D71, D72, D73, D8, D9: footprint kbd:D3_SMD_L1 -> kbd_Parts:Diode_SMD
- J1: footprint kbd:XH2.5_rev -> kbd_Parts:Battery_XH2.5_GL; moved to B.Cu
- L1, L10, L11, L12, L13, L14, L15, L16, L17, L18, L19, L2, L20, L21, L22, L23, L24, L25, L26, L27, L28, L29, L3, L30, L31, L32, L33, L34, L35, L36, L37, L38, L39, L4, L40, L41, L42, L43, L44, L45, L46, L47, L48, L49, L5, L50, L51, L52, L53, L54, L55, L56, L57, L58, L59, L6, L60, L61, L62, L63, L64, L65, L66, L67, L68, L69, L7, L70, L71, L72, L73, L8, L9: footprint kbd:YS-SK6812MINI-E_v3 -> kbd_Parts:LED_SK6812MINI-E_BL
- SW1, SW10, SW11, SW12, SW13, SW14, SW16, SW17, SW18, SW19, SW20, SW21, SW22, SW23, SW24, SW26, SW27, SW28, SW29, SW30, SW31, SW32, SW33, SW34, SW35, SW36, SW37, SW38, SW39, SW41, SW42, SW43, SW44, SW45, SW46, SW47, SW48, SW49, SW51, SW52, SW53, SW54, SW56, SW57, SW58, SW59, SW6, SW60, SW61, SW63, SW64, SW66, SW67, SW68, SW7, SW70, SW71, SW72, SW73, SW8, SW9: footprint kbd:CherryMX_Hotswap_BL_LH_v2 -> kbd_SW:CherryMX_Hotswap_1.0u
- SW15, SW25, SW40, SW5, SW50, SW55: footprint kbd:CherryMX_Hotswap_1.25u_LH_v2 -> kbd_SW:CherryMX_Hotswap_1.25u
- SW2: footprint kbd:CherryMX_Hotswap_1.5u_BL_LH_v2 -> kbd_SW:CherryMX_Hotswap_1.5u
- SW3, SW62: footprint kbd:CherryMX_Hotswap_1.75u_BL_LH_v2 -> kbd_SW:CherryMX_Hotswap_1.75u
- SW4: footprint kbd:CherryMX_Hotswap_2.25u_BL_v2 -> kbd_SW:CherryMX_Hotswap_2u
- SW65, SW69: footprint kbd:CherryMX_Hotswap_BL_LH_v2 -> kbd_SW:CherryMX_Hotswap_1.0u_Small1
- SW74: footprint kbd:ResetSW_FL -> kbd_Parts:ResetSW
- SW75: footprint kbd:Stab_2u_BL -> kbd_SW:CherryMX_stab_2u
- U1: footprint kbd:BLE_Micro_Pro_L1 -> kbd_Parts:Micon_BMP_GL
- turned J1 to 180 degrees
Routing:
- net VCC: track 2184.3 -> 2248.6 mm
- net Col6: track 398.8 -> 407.7 mm
- net Net-(D16-Pad2): track 36.2 -> 39.5 mm
- net Net-(D65-Pad1): track 29.3 -> 32.4 mm
- net Col4: track 386.5 -> 389.4 mm
- net Col5: track 494.9 -> 497.9 mm
- net Net-(D43-Pad1): track 28.3 -> 30.9 mm
- net Net-(D33-Pad2): track 34.3 -> 36.9 mm
- net Net-(D38-Pad1): track 26.7 -> 29.2 mm
- net Net-(D28-Pad2): track 35.9 -> 38.4 mm
- net Net-(D69-Pad1): track 39.6 -> 42.2 mm
- net Net-(D18-Pad2): track 33.8 -> 36.2 mm
- net Net-(D64-Pad1): track 26.7 -> 29.1 mm
- net Net-(D66-Pad1): track 16.7 -> 19.0 mm
- net Net-(D23-Pad2): track 34.2 -> 36.5 mm
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