File: KBD67mk2/1_Top/kbd67mk2_top.sch (KiCad schematic (older format))
At the start: 259 parts, among them J1 Conn_01x02, J10 Conn_01x01, J11 Conn_01x01, J12 Conn_01x01, J13 Conn_01x01, J14 Conn_01x01, J15 Conn_01x01, J16 Conn_01x01, J17 Conn_01x01, J2 Conn_01x01, J3 Conn_01x01, J4 Conn_01x01, J5 Conn_01x01, J6 Conn_01x01, J7 Conn_01x01, J8 Conn_01x01, J9 Conn_01x01, SW1 SW_PUSH, SW10 SW_PUSH, SW11 SW_PUSH, SW12 SW_PUSH, SW13 SW_PUSH, SW14 SW_PUSH, SW15 SW_PUSH, SW16 SW_PUSH, SW17 SW_PUSH, SW18 SW_PUSH, SW19 SW_PUSH, SW2 SW_PUSH, SW20 SW_PUSH, SW21 SW_PUSH, SW22 SW_PUSH, SW23 SW_PUSH, SW24 SW_PUSH, SW25 SW_PUSH, SW26 SW_PUSH, SW27 SW_PUSH, SW28 SW_PUSH, SW29 SW_PUSH, SW3 SW_PUSH, SW30 SW_PUSH, SW31 SW_PUSH, SW32 SW_PUSH, SW33 SW_PUSH, SW34 SW_PUSH, SW35 SW_PUSH, SW36 SW_PUSH, SW37 SW_PUSH, SW38 SW_PUSH, SW39 SW_PUSH, SW4 SW_PUSH, SW40 SW_PUSH, SW41 SW_PUSH, SW42 SW_PUSH, SW43 SW_PUSH, SW44 SW_PUSH, SW45 SW_PUSH, SW46 SW_PUSH, SW47 SW_PUSH, SW48 SW_PUSH, SW49 SW_PUSH, SW5 SW_PUSH, SW50 SW_PUSH, SW51 SW_PUSH, SW52 SW_PUSH, SW53 SW_PUSH, SW54 SW_PUSH, SW55 SW_PUSH, SW56 SW_PUSH, SW57 SW_PUSH, SW58 SW_PUSH, SW59 SW_PUSH, SW6 SW_PUSH, SW60 SW_PUSH, SW61 SW_PUSH, SW62 SW_PUSH, SW63 SW_PUSH, SW64 SW_PUSH, SW65 SW_PUSH, SW66 SW_PUSH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

Commit message: いっぱい追加
Parts:
- D1, D10, D11, D12, D13, D14, D15, D16, D17, D18, D19, D2, D20, D21, D22, D23, D24, D25, D26, D27, D28, D29, D3, D30, D31, D32, D33, D34, D35, D36, D37, D38, D39, D4, D40, D41, D42, D43, D44, D45, D46, D47, D48, D49, D5, D50, D51, D52, D53, D54, D55, D56, D57, D58, D59, D6, D60, D61, D62, D63, D64, D65, D66, D67, D68, D69, D7, D70, D71, D72, D73, D74, D75, D76, D77, D78, D79, D8, D80, D9: footprint kbd_Parts:Diode_TH_SMD -> kbd:D3_TH_SMD_BL
- J1: footprint kbd_Parts:Battery_XH2.5_GL -> kbd:XH2.5_rev
- J10, J11, J12, J13, J14, J15, J16, J17, J8, J9: footprint kbd_Hole:m2_Screw_Hole_Fab -> kbd:HOLE_m2_Outline_Fab
- J2, J3, J4, J5, J6, J7: footprint kbd_Hole:m2_Screw_Hole_EdgeCuts -> kbd:HOLE_m2_Outline
- L1: footprint kbd_Parts:LED_SK6812MINI-E_BL -> kbd:YS-SK6812MINI-E_v3
- L10: renamed from L23; footprint kbd_Parts:LED_SK6812MINI-E_BL -> kbd:YS-SK6812MINI-E_v3
- L11: renamed from L63; footprint kbd_Parts:LED_SK6812MINI-E_BL -> kbd:YS-SK6812MINI-E_v3
- L12: renamed from L43; footprint kbd_Parts:LED_SK6812MINI-E_BL -> kbd:YS-SK6812MINI-E_v3
- L13: renamed from L4; footprint kbd_Parts:LED_SK6812MINI-E_BL -> kbd:YS-SK6812MINI-E_v3
- L14: renamed from L24; footprint kbd_Parts:LED_SK6812MINI-E_BL -> kbd:YS-SK6812MINI-E_v3
- L15: renamed from L64; footprint kbd_Parts:LED_SK6812MINI-E_BL -> kbd:YS-SK6812MINI-E_v3
- L16: renamed from L44; footprint kbd_Parts:LED_SK6812MINI-E_BL -> kbd:YS-SK6812MINI-E_v3
- L17: renamed from L5; footprint kbd_Parts:LED_SK6812MINI-E_BL -> kbd:YS-SK6812MINI-E_v3
- L18: renamed from L25; footprint kbd_Parts:LED_SK6812MINI-E_BL -> kbd:YS-SK6812MINI-E_v3
- L19: renamed from L65; footprint kbd_Parts:LED_SK6812MINI-E_BL -> kbd:YS-SK6812MINI-E_v3
- L2: renamed from L21; footprint kbd_Parts:LED_SK6812MINI-E_BL -> kbd:YS-SK6812MINI-E_v3
- L20: renamed from L45; footprint kbd_Parts:LED_SK6812MINI-E_BL -> kbd:YS-SK6812MINI-E_v3
- L21: renamed from L6; footprint kbd_Parts:LED_SK6812MINI-E_BL -> kbd:YS-SK6812MINI-E_v3
- L22: renamed from L26; footprint kbd_Parts:LED_SK6812MINI-E_BL -> kbd:YS-SK6812MINI-E_v3
- L23: renamed from L66; footprint kbd_Parts:LED_SK6812MINI-E_BL -> kbd:YS-SK6812MINI-E_v3
- L24: renamed from L46; footprint kbd_Parts:LED_SK6812MINI-E_BL -> kbd:YS-SK6812MINI-E_v3
- L25: renamed from L7; footprint kbd_Parts:LED_SK6812MINI-E_BL -> kbd:YS-SK6812MINI-E_v3
- L26: renamed from L27; footprint kbd_Parts:LED_SK6812MINI-E_BL -> kbd:YS-SK6812MINI-E_v3
- L27: renamed from L67; footprint kbd_Parts:LED_SK6812MINI-E_BL -> kbd:YS-SK6812MINI-E_v3
- L28: renamed from L47; footprint kbd_Parts:LED_SK6812MINI-E_BL -> kbd:YS-SK6812MINI-E_v3
- L29: renamed from L8; footprint kbd_Parts:LED_SK6812MINI-E_BL -> kbd:YS-SK6812MINI-E_v3
- L3: renamed from L61; footprint kbd_Parts:LED_SK6812MINI-E_BL -> kbd:YS-SK6812MINI-E_v3
- L30: renamed from L28; footprint kbd_Parts:LED_SK6812MINI-E_BL -> kbd:YS-SK6812MINI-E_v3
- L31: renamed from L68; footprint kbd_Parts:LED_SK6812MINI-E_BL -> kbd:YS-SK6812MINI-E_v3
- L32: renamed from L48; footprint kbd_Parts:LED_SK6812MINI-E_BL -> kbd:YS-SK6812MINI-E_v3
- L33: renamed from L9; footprint kbd_Parts:LED_SK6812MINI-E_BL -> kbd:YS-SK6812MINI-E_v3
- L34: renamed from L29; footprint kbd_Parts:LED_SK6812MINI-E_BL -> kbd:YS-SK6812MINI-E_v3
- L35: renamed from L69; footprint kbd_Parts:LED_SK6812MINI-E_BL -> kbd:YS-SK6812MINI-E_v3
- L36: renamed from L49; footprint kbd_Parts:LED_SK6812MINI-E_BL -> kbd:YS-SK6812MINI-E_v3
- L37: renamed from L10; footprint kbd_Parts:LED_SK6812MINI-E_BL -> kbd:YS-SK6812MINI-E_v3
- L38: renamed from L30; footprint kbd_Parts:LED_SK6812MINI-E_BL -> kbd:YS-SK6812MINI-E_v3
- L39: renamed from L70; footprint kbd_Parts:LED_SK6812MINI-E_BL -> kbd:YS-SK6812MINI-E_v3
- L4: renamed from L41; footprint kbd_Parts:LED_SK6812MINI-E_BL -> kbd:YS-SK6812MINI-E_v3
- L40: renamed from L50; footprint kbd_Parts:LED_SK6812MINI-E_BL -> kbd:YS-SK6812MINI-E_v3
- L41: renamed from L11; footprint kbd_Parts:LED_SK6812MINI-E_BL -> kbd:YS-SK6812MINI-E_v3
- L42: renamed from L31; footprint kbd_Parts:LED_SK6812MINI-E_BL -> kbd:YS-SK6812MINI-E_v3
- L43: renamed from L71; footprint kbd_Parts:LED_SK6812MINI-E_BL -> kbd:YS-SK6812MINI-E_v3
- L44: renamed from L51; footprint kbd_Parts:LED_SK6812MINI-E_BL -> kbd:YS-SK6812MINI-E_v3
- L45: renamed from L12; footprint kbd_Parts:LED_SK6812MINI-E_BL -> kbd:YS-SK6812MINI-E_v3
- L46: renamed from L32; footprint kbd_Parts:LED_SK6812MINI-E_BL -> kbd:YS-SK6812MINI-E_v3
- L47: renamed from L72; footprint kbd_Parts:LED_SK6812MINI-E_BL -> kbd:YS-SK6812MINI-E_v3
- L48: renamed from L52; footprint kbd_Parts:LED_SK6812MINI-E_BL -> kbd:YS-SK6812MINI-E_v3
- L49: renamed from L13; footprint kbd_Parts:LED_SK6812MINI-E_BL -> kbd:YS-SK6812MINI-E_v3
- L5: renamed from L2; footprint kbd_Parts:LED_SK6812MINI-E_BL -> kbd:YS-SK6812MINI-E_v3
- L50: renamed from L33; footprint kbd_Parts:LED_SK6812MINI-E_BL -> kbd:YS-SK6812MINI-E_v3
- L51: renamed from L73; footprint kbd_Parts:LED_SK6812MINI-E_BL -> kbd:YS-SK6812MINI-E_v3
- L52: renamed from L53; footprint kbd_Parts:LED_SK6812MINI-E_BL -> kbd:YS-SK6812MINI-E_v3
- L53: renamed from L14; footprint kbd_Parts:LED_SK6812MINI-E_BL -> kbd:YS-SK6812MINI-E_v3
- L54: renamed from L34; footprint kbd_Parts:LED_SK6812MINI-E_BL -> kbd:YS-SK6812MINI-E_v3
- L55: renamed from L74; footprint kbd_Parts:LED_SK6812MINI-E_BL -> kbd:YS-SK6812MINI-E_v3
- L56: renamed from L54; footprint kbd_Parts:LED_SK6812MINI-E_BL -> kbd:YS-SK6812MINI-E_v3
- L57: renamed from L15; footprint kbd_Parts:LED_SK6812MINI-E_BL -> kbd:YS-SK6812MINI-E_v3
- L58: renamed from L35; footprint kbd_Parts:LED_SK6812MINI-E_BL -> kbd:YS-SK6812MINI-E_v3
- L59: renamed from L75; footprint kbd_Parts:LED_SK6812MINI-E_BL -> kbd:YS-SK6812MINI-E_v3
- L6: renamed from L22; footprint kbd_Parts:LED_SK6812MINI-E_BL -> kbd:YS-SK6812MINI-E_v3
- L60: renamed from L55; footprint kbd_Parts:LED_SK6812MINI-E_BL -> kbd:YS-SK6812MINI-E_v3
- L61: renamed from L16; footprint kbd_Parts:LED_SK6812MINI-E_BL -> kbd:YS-SK6812MINI-E_v3
- L62: renamed from L36; footprint kbd_Parts:LED_SK6812MINI-E_BL -> kbd:YS-SK6812MINI-E_v3
- L63: renamed from L76; footprint kbd_Parts:LED_SK6812MINI-E_BL -> kbd:YS-SK6812MINI-E_v3
- L64: renamed from L56; footprint kbd_Parts:LED_SK6812MINI-E_BL -> kbd:YS-SK6812MINI-E_v3
- L65: renamed from L17; footprint kbd_Parts:LED_SK6812MINI-E_BL -> kbd:YS-SK6812MINI-E_v3
- L66: renamed from L37; footprint kbd_Parts:LED_SK6812MINI-E_BL -> kbd:YS-SK6812MINI-E_v3
- L67: renamed from L77; footprint kbd_Parts:LED_SK6812MINI-E_BL -> kbd:YS-SK6812MINI-E_v3
- L68: renamed from L57; footprint kbd_Parts:LED_SK6812MINI-E_BL -> kbd:YS-SK6812MINI-E_v3
- L69: renamed from L18; footprint kbd_Parts:LED_SK6812MINI-E_BL -> kbd:YS-SK6812MINI-E_v3
- L7: renamed from L62; footprint kbd_Parts:LED_SK6812MINI-E_BL -> kbd:YS-SK6812MINI-E_v3
- L70: renamed from L38; footprint kbd_Parts:LED_SK6812MINI-E_BL -> kbd:YS-SK6812MINI-E_v3
- L71: renamed from L78; footprint kbd_Parts:LED_SK6812MINI-E_BL -> kbd:YS-SK6812MINI-E_v3
- L72: renamed from L58; footprint kbd_Parts:LED_SK6812MINI-E_BL -> kbd:YS-SK6812MINI-E_v3
- L73: renamed from L19; footprint kbd_Parts:LED_SK6812MINI-E_BL -> kbd:YS-SK6812MINI-E_v3
- L74: renamed from L39; footprint kbd_Parts:LED_SK6812MINI-E_BL -> kbd:YS-SK6812MINI-E_v3
- L75: renamed from L79; footprint kbd_Parts:LED_SK6812MINI-E_BL -> kbd:YS-SK6812MINI-E_v3
- L76: renamed from L59; footprint kbd_Parts:LED_SK6812MINI-E_BL -> kbd:YS-SK6812MINI-E_v3
- L77: renamed from L20; footprint kbd_Parts:LED_SK6812MINI-E_BL -> kbd:YS-SK6812MINI-E_v3
- L78: renamed from L40; footprint kbd_Parts:LED_SK6812MINI-E_BL -> kbd:YS-SK6812MINI-E_v3
- L79: renamed from L80; footprint kbd_Parts:LED_SK6812MINI-E_BL -> kbd:YS-SK6812MINI-E_v3
- L8: renamed from L42; footprint kbd_Parts:LED_SK6812MINI-E_BL -> kbd:YS-SK6812MINI-E_v3
- L80: renamed from L60; footprint kbd_Parts:LED_SK6812MINI-E_BL -> kbd:YS-SK6812MINI-E_v3
- L9: renamed from L3; footprint kbd_Parts:LED_SK6812MINI-E_BL -> kbd:YS-SK6812MINI-E_v3
- SW1, SW10, SW11, SW12, SW13, SW14, SW15, SW16, SW17, SW18, SW19, SW2, SW20, SW21, SW22, SW23, SW24, SW25, SW26, SW27, SW28, SW29, SW3, SW30, SW31, SW32, SW33, SW34, SW35, SW36, SW37, SW38, SW39, SW4, SW40, SW41, SW42, SW43, SW44, SW45, SW46, SW47, SW48, SW49, SW5, SW50, SW51, SW52, SW53, SW54, SW55, SW56, SW57, SW58, SW59, SW6, SW60, SW61, SW62, SW63, SW64, SW65, SW66, SW67, SW68, SW69, SW7, SW70, SW71, SW72, SW73, SW74, SW75, SW76, SW77, SW78, SW79, SW8, SW80, SW9: footprint kbd_SW:CherryMX_Choc_Hotswap_1u -> kbd:CherryMX_Choc_Hotswap_LH_v2
- SW81: footprint kbd_Parts:ResetSW -> kbd:ResetSW
- U1: footprint kbd_Parts:Micon_BMP_GL -> kbd:BLE_Micro_Pro_L1
Connections:
- net at L3.3 (DIN): now also L78.1 (DOUT); no longer L80.1 (DOUT)
- net at L4.3 (DIN): now also L79.1 (DOUT); no longer L78.1 (DOUT)
Other:
- note added: "Left hand block (Max 35 keys)"
- note added: "Right hand block (Max 35 keys)"
- note removed: "Left hand block (Max 40 keys)"
- note removed: "Right hand block (Max 40 keys)"
- moved on the sheet: L1, L10, L11, L12, L13, L14, L15, L16, L17, L18, L19, L2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
