File: Keyboard/KBD67mk2/1_Top_TH/kbd67mk2_top.kicad_pcb (KiCad board)
At the start: 2 copper layers, 315.8 x 99.2 mm, 84 parts, among them J10 Conn_01x01, J11 Conn_01x01, J12 Conn_01x01, J13 Conn_01x01, J14 Conn_01x01, J15 Conn_01x01, J16 Conn_01x01, J17 Conn_01x01, J2 Conn_01x01, J3 Conn_01x01, J4 Conn_01x01, J5 Conn_01x01, J6 Conn_01x01, J7 Conn_01x01, J8 Conn_01x01, J9 Conn_01x01, SW1 SW_PUSH, SW2 KEY_SWITCH, SW3 SW_PUSH, SW4 KEY_SWITCH, SW4 SW_PUSH, SW5 SW_PUSH, SW7 SW_PUSH, SW8 SW_PUSH

Commit message: 寸法更新とか
Other:
- board size 315.8 x 99.2 mm -> 314.4 x 98.8 mm
Changed lines of the file:
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@@
   (general
     (thickness 1.6)
-    (drawings 52)
+    (drawings 54)
     (tracks 0)
     (zones 0)
@@
     (pad 1 thru_hole oval (at 0 -7 90) (size 2 15.9) (drill oval 0.3 14.2) (layers *.Cu *.Mask))
   )
+  (gr_line (start 329.325 113.75) (end 329.325 19.55) (layer F.Fab) (width 0.15))
+  (gr_line (start 13.575 113.75) (end 13.575 19.55) (layer F.Fab) (width 0.15))
   (dimension 2.5 (width 0.15) (layer Dwgs.User)
     (gr_text "2.500 mm" (at 14.85 108.85) (layer Dwgs.User)
@@
   (gr_line (start 78.575 20.55) (end 264.325 20.55) (layer F.Fab) (width 0.15))
   (gr_line (start 10.45 50.55) (end 332.4 50.55) (layer F.Fab) (width 0.15))
-  (gr_arc (start 320.825 20.05) (end 323.825 20.05) (angle -90) (layer F.Fab) (width 0.1))
-  (gr_arc (start 320.825 113.25) (end 320.825 116.25) (angle -90) (layer F.Fab) (width 0.1))
-  (gr_arc (start 22.075 20.05) (end 22.075 17.05) (angle -90) (layer F.Fab) (width 0.1))
-  (gr_arc (start 22.075 113.25) (end 19.075 113.25) (angle -90) (layer F.Fab) (width 0.1))
+  (gr_arc (start 320.625 20.25) (end 323.625 20.25) (angle -90) (layer F.Fab) (width 0.1))
+  (gr_arc (start 320.625 113.05) (end 320.625 116.05) (angle -90) (layer F.Fab) (width 0.1))
+  (gr_arc (start 22.275 20.25) (end 22.275 17.25) (angle -90) (layer F.Fab) (width 0.1))
+  (gr_arc (start 22.275 113.05) (end 19.275 113.05) (angle -90) (layer F.Fab) (width 0.1))
   (gr_text "Do not place switches to the left of this line." (at 32.5 13.7) (layer F.Fab)
     (effects (font (size 1 1) (thickness 0.15)))
@@
     (effects (font (size 1 1) (thickness 0.15)))
   )
-  (gr_line (start 323.825 20.05) (end 323.825 113.25) (layer F.Fab) (width 0.1))
-  (gr_line (start 19.075 20.05) (end 19.075 113.25) (layer F.Fab) (width 0.1))
-  (gr_arc (start 16.575 113.25) (end 13.575 113.25) (angle -90) (layer Edge.Cuts) (width 0.1))
-  (gr_arc (start 16.575 20.05) (end 16.575 17.05) (angle -90) (layer Edge.Cuts) (width 0.1))
-  (gr_arc (start 326.325 20.05) (end 329.325 20.05) (angle -90) (layer Edge.Cuts) (width 0.1))
-  (gr_arc (start 326.325 113.25) (end 326.325 116.25) (angle -90) (layer Edge.Cuts) (width 0.1))
-  (gr_line (start 329.325 113.25) (end 329.325 20.05) (layer Edge.Cuts) (width 0.1))
-  (gr_line (start 16.575 116.25) (end 326.325 116.25) (layer Edge.Cuts) (width 0.1))
-  (gr_line (start 13.575 20.05) (end 13.575 113.25) (layer Edge.Cuts) (width 0.1))
-  (gr_line (start 326.325 17.05) (end 16.575 17.05) (layer Edge.Cuts) (width 0.1))
+  (gr_line (start 323.625 20.25) (end 323.625 113.05) (layer F.Fab) (width 0.1))
+  (gr_line (start 19.275 20.25) (end 19.275 113.05) (layer F.Fab) (width 0.1))
+  (gr_arc (start 17.275 113.05) (end 14.275 113.05) (angle -90) (layer Edge.Cuts) (width 0.1))
+  (gr_arc (start 17.275 20.25) (end 17.275 17.25) (angle -90) (layer Edge.Cuts) (width 0.1))
+  (gr_arc (start 325.625 20.25) (end 328.625 20.25) (angle -90) (layer Edge.Cuts) (width 0.1))
+  (gr_arc (start 325.625 113.05) (end 325.625 116.05) (angle -90) (layer Edge.Cuts) (width 0.1))
+  (gr_line (start 328.625 113.05) (end 328.625 20.25) (layer Edge.Cuts) (width 0.1))
+  (gr_line (start 17.275 116.05) (end 325.625 116.05) (layer Edge.Cuts) (width 0.1))
+  (gr_line (start 14.275 20.25) (end 14.275 113.05) (layer Edge.Cuts) (width 0.1))
+  (gr_line (start 325.625 17.25) (end 17.275 17.25) (layer Edge.Cuts) (width 0.1))
   (zone (net 0) (net_name "") (layer F.Cu) (hatch edge 0.508)
     (connect_pads (clearance 0.508))
