File: Parts/BottomPlate/Blank/65BlankBottom.kicad_pcb (KiCad board)
At the start: 2 copper layers, 325.8 x 41.2 mm, 4 parts

Commit message: 諸々修正
今度はちゃんと説明書きを書く
Parts:
- added Ref**: Val**, kbd:HOLE_m2_a, F.Cu at (178.4, 26.0)
- added Ref**: Val**, kbd:HOLE_m2_a, F.Cu at (178.4, 55.2)
Other:
- board size 325.8 x 41.2 mm -> 323.8 x 41.2 mm
