File: Parts/BackPlate/Blank/65BlankBack.kicad_pcb (KiCad board)
At the start: 2 copper layers, 172.9 x 20 mm, 3 parts

Commit message: 寸法更新とか
Other:
- board size 172.9 x 20 mm -> 172.9 x 19.4 mm
Changed lines of the file:
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@@
     (arrow2b (pts (xy 10.925 20) (xy 11.511421 21.126504)))
   )
-  (gr_line (start 14 40) (end 166.875 40) (layer Edge.Cuts) (width 0.1))
-  (gr_line (start 14 20) (end 186.875 20) (layer Edge.Cuts) (width 0.1))
+  (gr_line (start 14 39.7) (end 166.875 39.7) (layer Edge.Cuts) (width 0.1))
+  (gr_line (start 14 20.3) (end 186.875 20.3) (layer Edge.Cuts) (width 0.1))
   (gr_arc (start 183.875 27) (end 183.875 30) (angle -90) (layer Edge.Cuts) (width 0.1))
   (gr_arc (start 169.875 33) (end 169.875 30) (angle -90) (layer Edge.Cuts) (width 0.1))
-  (gr_line (start 186.875 27) (end 186.875 20) (layer Edge.Cuts) (width 0.1))
+  (gr_line (start 186.875 27) (end 186.875 20.3) (layer Edge.Cuts) (width 0.1))
   (gr_line (start 169.875 30) (end 183.875 30) (layer Edge.Cuts) (width 0.1))
-  (gr_line (start 166.875 40) (end 166.875 33) (layer Edge.Cuts) (width 0.1))
-  (gr_line (start 14 20) (end 14 40) (layer Edge.Cuts) (width 0.1))
+  (gr_line (start 166.875 39.7) (end 166.875 33) (layer Edge.Cuts) (width 0.1))
+  (gr_line (start 14 20.3) (end 14 39.7) (layer Edge.Cuts) (width 0.1))
   (zone (net 0) (net_name "") (layer F.Cu) (hatch edge 0.508)
     (connect_pads (clearance 0.508))

Commit message: 諸々修正
今度はちゃんと説明書きを書く
Other:
- board size 172.9 x 19.4 mm -> 171.9 x 19.4 mm
Changed lines of the file:
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@@
-(kicad_pcb (version 20171130) (host pcbnew "(5.1.5)-3")
+(kicad_pcb (version 20171130) (host pcbnew "(5.1.10)-1")
   (general
     (thickness 1.6)
@@
     (pad_drill 0)
     (pad_to_mask_clearance 0)
-    (solder_mask_min_width 0.25)
     (aux_axis_origin 47.625 47.625)
     (grid_origin 47.625 47.625)
@@
     (pad "" np_thru_hole circle (at 0 0) (size 2.2 2.2) (drill 2.2) (layers *.Cu *.Mask))
   )
-  (dimension 172.875 (width 0.15) (layer F.Fab)
-    (gr_text "172.875 mm" (at 100.4375 16.025) (layer F.Fab)
+  (dimension 171.875 (width 0.15) (layer F.Fab)
+    (gr_text "171.875 mm" (at 100.9375 16.325) (layer F.Fab)
       (effects (font (size 1 1) (thickness 0.15)))
     )
-    (feature1 (pts (xy 186.875 20) (xy 186.875 16.738579)))
-    (feature2 (pts (xy 14 20) (xy 14 16.738579)))
-    (crossbar (pts (xy 14 17.325) (xy 186.875 17.325)))
-    (arrow1a (pts (xy 186.875 17.325) (xy 185.748496 17.911421)))
-    (arrow1b (pts (xy 186.875 17.325) (xy 185.748496 16.738579)))
-    (arrow2a (pts (xy 14 17.325) (xy 15.126504 17.911421)))
-    (arrow2b (pts (xy 14 17.325) (xy 15.126504 16.738579)))
+    (feature1 (pts (xy 186.875 20.3) (xy 186.875 17.038579)))
+    (feature2 (pts (xy 15 20.3) (xy 15 17.038579)))
+    (crossbar (pts (xy 15 17.625) (xy 186.875 17.625)))
+    (arrow1a (pts (xy 186.875 17.625) (xy 185.748496 18.211421)))
+    (arrow1b (pts (xy 186.875 17.625) (xy 185.748496 17.038579)))
+    (arrow2a (pts (xy 15 17.625) (xy 16.126504 18.211421)))
+    (arrow2b (pts (xy 15 17.625) (xy 16.126504 17.038579)))
   )
-  (dimension 20 (width 0.15) (layer F.Fab)
-    (gr_text "20.000 mm" (at 9.625 30 270) (layer F.Fab)
+  (dimension 19.4 (width 0.15) (layer F.Fab)
+    (gr_text "19.400 mm" (at 10.625 30 270) (layer F.Fab)
       (effects (font (size 1 1) (thickness 0.15)))
     )
-    (feature1 (pts (xy 14 40) (xy 10.338579 40)))
-    (feature2 (pts (xy 14 20) (xy 10.338579 20)))
-    (crossbar (pts (xy 10.925 20) (xy 10.925 40)))
-    (arrow1a (pts (xy 10.925 40) (xy 10.338579 38.873496)))
-    (arrow1b (pts (xy 10.925 40) (xy 11.511421 38.873496)))
-    (arrow2a (pts (xy 10.925 20) (xy 10.338579 21.126504)))
-    (arrow2b (pts (xy 10.925 20) (xy 11.511421 21.126504)))
+    (feature1 (pts (xy 15 39.7) (xy 11.338579 39.7)))
+    (feature2 (pts (xy 15 20.3) (xy 11.338579 20.3)))
+    (crossbar (pts (xy 11.925 20.3) (xy 11.925 39.7)))
+    (arrow1a (pts (xy 11.925 39.7) (xy 11.338579 38.573496)))
+    (arrow1b (pts (xy 11.925 39.7) (xy 12.511421 38.573496)))
+    (arrow2a (pts (xy 11.925 20.3) (xy 11.338579 21.426504)))
+    (arrow2b (pts (xy 11.925 20.3) (xy 12.511421 21.426504)))
   )
-  (gr_line (start 14 39.7) (end 166.875 39.7) (layer Edge.Cuts) (width 0.1))
-  (gr_line (start 14 20.3) (end 186.875 20.3) (layer Edge.Cuts) (width 0.1))
+  (gr_line (start 15 39.7) (end 166.875 39.7) (layer Edge.Cuts) (width 0.1))
+  (gr_line (start 15 20.3) (end 186.875 20.3) (layer Edge.Cuts) (width 0.1))
   (gr_arc (start 183.875 27) (end 183.875 30) (angle -90) (layer Edge.Cuts) (width 0.1))
   (gr_arc (start 169.875 33) (end 169.875 30) (angle -90) (layer Edge.Cuts) (width 0.1))
@@
   (gr_line (start 169.875 30) (end 183.875 30) (layer Edge.Cuts) (width 0.1))
   (gr_line (start 166.875 39.7) (end 166.875 33) (layer Edge.Cuts) (width 0.1))
-  (gr_line (start 14 20.3) (end 14 39.7) (layer Edge.Cuts) (width 0.1))
+  (gr_line (start 15 20.3) (end 15 39.7) (layer Edge.Cuts) (width 0.1))
   (zone (net 0) (net_name "") (layer F.Cu) (hatch edge 0.508)
     (connect_pads (clearance 0.508))

Commit message: ケース修正に伴う修正
Other:
- board size 171.9 x 19.4 mm -> 171.4 x 19.4 mm
Changed lines of the file:
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@@
       (effects (font (size 1 1) (thickness 0.15)))
     )
+    (fp_circle (center 0 0) (end 2.2 0) (layer Cmts.User) (width 0.15))
     (fp_circle (center 0 0) (end 2.45 0) (layer F.CrtYd) (width 0.05))
-    (fp_circle (center 0 0) (end 2.2 0) (layer Cmts.User) (width 0.15))
     (fp_text user %R (at 0.3 0) (layer F.Fab) hide
       (effects (font (size 1 1) (thickness 0.15)))
@@
       (effects (font (size 1 1) (thickness 0.15)))
     )
+    (fp_circle (center 0 0) (end 2.2 0) (layer Cmts.User) (width 0.15))
     (fp_circle (center 0 0) (end 2.45 0) (layer F.CrtYd) (width 0.05))
-    (fp_circle (center 0 0) (end 2.2 0) (layer Cmts.User) (width 0.15))
     (fp_text user %R (at 0.3 0) (layer F.Fab) hide
       (effects (font (size 1 1) (thickness 0.15)))
@@
       (effects (font (size 1 1) (thickness 0.15)))
     )
+    (fp_circle (center 0 0) (end 2.2 0) (layer Cmts.User) (width 0.15))
     (fp_circle (center 0 0) (end 2.45 0) (layer F.CrtYd) (width 0.05))
-    (fp_circle (center 0 0) (end 2.2 0) (layer Cmts.User) (width 0.15))
     (fp_text user %R (at 0.3 0) (layer F.Fab) hide
       (effects (font (size 1 1) (thickness 0.15)))
@@
     (pad "" np_thru_hole circle (at 0 0) (size 2.2 2.2) (drill 2.2) (layers *.Cu *.Mask))
   )
-  (dimension 171.875 (width 0.15) (layer F.Fab)
-    (gr_text "171.875 mm" (at 100.9375 16.325) (layer F.Fab)
+  (dimension 171.375 (width 0.15) (layer F.Fab)
+    (gr_text "171.375 mm" (at 101.1875 16.325) (layer F.Fab)
       (effects (font (size 1 1) (thickness 0.15)))
     )
     (feature1 (pts (xy 186.875 20.3) (xy 186.875 17.038579)))
-    (feature2 (pts (xy 15 20.3) (xy 15 17.038579)))
-    (crossbar (pts (xy 15 17.625) (xy 186.875 17.625)))
+    (feature2 (pts (xy 15.5 20.3) (xy 15.5 17.038579)))
+    (crossbar (pts (xy 15.5 17.625) (xy 186.875 17.625)))
     (arrow1a (pts (xy 186.875 17.625) (xy 185.748496 18.211421)))
     (arrow1b (pts (xy 186.875 17.625) (xy 185.748496 17.038579)))
-    (arrow2a (pts (xy 15 17.625) (xy 16.126504 18.211421)))
-    (arrow2b (pts (xy 15 17.625) (xy 16.126504 17.038579)))
+    (arrow2a (pts (xy 15.5 17.625) (xy 16.626504 18.211421)))
+    (arrow2b (pts (xy 15.5 17.625) (xy 16.626504 17.038579)))
   )
   (dimension 19.4 (width 0.15) (layer F.Fab)
-    (gr_text "19.400 mm" (at 10.625 30 270) (layer F.Fab)
+    (gr_text "19.400 mm" (at 11.125 30 270) (layer F.Fab)
       (effects (font (size 1 1) (thickness 0.15)))
     )
-    (feature1 (pts (xy 15 39.7) (xy 11.338579 39.7)))
-    (feature2 (pts (xy 15 20.3) (xy 11.338579 20.3)))
-    (crossbar (pts (xy 11.925 20.3) (xy 11.925 39.7)))
-    (arrow1a (pts (xy 11.925 39.7) (xy 11.338579 38.573496)))
-    (arrow1b (pts (xy 11.925 39.7) (xy 12.511421 38.573496)))
-    (arrow2a (pts (xy 11.925 20.3) (xy 11.338579 21.426504)))
-    (arrow2b (pts (xy 11.925 20.3) (xy 12.511421 21.426504)))
+    (feature1 (pts (xy 15.5 39.7) (xy 11.838579 39.7)))
+    (feature2 (pts (xy 15.5 20.3) (xy 11.838579 20.3)))
+    (crossbar (pts (xy 12.425 20.3) (xy 12.425 39.7)))
+    (arrow1a (pts (xy 12.425 39.7) (xy 11.838579 38.573496)))
+    (arrow1b (pts (xy 12.425 39.7) (xy 13.011421 38.573496)))
+    (arrow2a (pts (xy 12.425 20.3) (xy 11.838579 21.426504)))
+    (arrow2b (pts (xy 12.425 20.3) (xy 13.011421 21.426504)))
   )
-  (gr_line (start 15 39.7) (end 166.875 39.7) (layer Edge.Cuts) (width 0.1))
-  (gr_line (start 15 20.3) (end 186.875 20.3) (layer Edge.Cuts) (width 0.1))
+  (gr_line (start 15.5 39.7) (end 166.875 39.7) (layer Edge.Cuts) (width 0.1))
+  (gr_line (start 15.5 20.3) (end 186.875 20.3) (layer Edge.Cuts) (width 0.1))
   (gr_arc (start 183.875 27) (end 183.875 30) (angle -90) (layer Edge.Cuts) (width 0.1))
   (gr_arc (start 169.875 33) (end 169.875 30) (angle -90) (layer Edge.Cuts) (width 0.1))
@@
   (gr_line (start 169.875 30) (end 183.875 30) (layer Edge.Cuts) (width 0.1))
   (gr_line (start 166.875 39.7) (end 166.875 33) (layer Edge.Cuts) (width 0.1))
-  (gr_line (start 15 20.3) (end 15 39.7) (layer Edge.Cuts) (width 0.1))
+  (gr_line (start 15.5 20.3) (end 15.5 39.7) (layer Edge.Cuts) (width 0.1))
   (zone (net 0) (net_name "") (layer F.Cu) (hatch edge 0.508)
     (connect_pads (clearance 0.508))
