File: Parts/BackPlate/CableHole/65CableHole.kicad_pcb (KiCad board)
At the start: 2 copper layers, 172.9 x 20 mm, 3 parts

Commit message: 寸法更新とか
Other:
- board size 172.9 x 20 mm -> 172.9 x 19.4 mm
Changed lines of the file:
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@@
     (arrow2b (pts (xy 339.75 45.24375) (xy 338.623496 45.830171)))
   )
-  (gr_line (start 186.875 20) (end 339.75 20) (layer Edge.Cuts) (width 0.1))
+  (gr_line (start 186.875 20.3) (end 339.75 20.3) (layer Edge.Cuts) (width 0.1))
   (gr_line (start 172.875 33) (end 172.875 30) (layer Edge.Cuts) (width 0.1))
   (gr_arc (start 169.875 33) (end 169.875 36) (angle -90) (layer Edge.Cuts) (width 0.1))
   (gr_line (start 169.875 36) (end 166.875 36) (layer Edge.Cuts) (width 0.1))
   (gr_arc (start 183.875 27) (end 183.875 30) (angle -90) (layer Edge.Cuts) (width 0.1))
-  (gr_line (start 186.875 27) (end 186.875 20) (layer Edge.Cuts) (width 0.1))
+  (gr_line (start 186.875 27) (end 186.875 20.3) (layer Edge.Cuts) (width 0.1))
   (gr_line (start 172.875 30) (end 183.875 30) (layer Edge.Cuts) (width 0.1))
-  (gr_line (start 166.875 40) (end 166.875 36) (layer Edge.Cuts) (width 0.1))
-  (gr_line (start 339.75 40) (end 339.75 20) (layer Edge.Cuts) (width 0.1))
-  (gr_line (start 166.875 40) (end 339.75 40) (layer Edge.Cuts) (width 0.1))
+  (gr_line (start 166.875 39.7) (end 166.875 36) (layer Edge.Cuts) (width 0.1))
+  (gr_line (start 339.75 39.7) (end 339.75 20.3) (layer Edge.Cuts) (width 0.1))
+  (gr_line (start 166.875 39.7) (end 339.75 39.7) (layer Edge.Cuts) (width 0.1))
   (zone (net 0) (net_name "") (layer F.Cu) (hatch edge 0.508)
     (connect_pads (clearance 0.508))

Commit message: 諸々修正
今度はちゃんと説明書きを書く
Other:
- board size 172.9 x 19.4 mm -> 171.9 x 19.4 mm
Changed lines of the file:
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@@
-(kicad_pcb (version 20171130) (host pcbnew "(5.1.5)-3")
+(kicad_pcb (version 20171130) (host pcbnew "(5.1.10)-1")
   (general
     (thickness 1.6)
@@
     (pad_drill 0)
     (pad_to_mask_clearance 0)
-    (solder_mask_min_width 0.25)
     (aux_axis_origin 47.625 47.625)
     (grid_origin 47.625 47.625)
@@
       (effects (font (size 1 1) (thickness 0.15)))
     )
+    (fp_circle (center 0 0) (end 2.2 0) (layer Cmts.User) (width 0.15))
     (fp_circle (center 0 0) (end 2.45 0) (layer F.CrtYd) (width 0.05))
-    (fp_circle (center 0 0) (end 2.2 0) (layer Cmts.User) (width 0.15))
     (fp_text user %R (at 0.3 0) (layer F.Fab) hide
       (effects (font (size 1 1) (thickness 0.15)))
@@
       (effects (font (size 1 1) (thickness 0.15)))
     )
+    (fp_circle (center 0 0) (end 2.2 0) (layer Cmts.User) (width 0.15))
     (fp_circle (center 0 0) (end 2.45 0) (layer F.CrtYd) (width 0.05))
-    (fp_circle (center 0 0) (end 2.2 0) (layer Cmts.User) (width 0.15))
     (fp_text user %R (at 0.3 0) (layer F.Fab) hide
       (effects (font (size 1 1) (thickness 0.15)))
@@
       (effects (font (size 1 1) (thickness 0.15)))
     )
+    (fp_circle (center 0 0) (end 2.2 0) (layer Cmts.User) (width 0.15))
     (fp_circle (center 0 0) (end 2.45 0) (layer F.CrtYd) (width 0.05))
-    (fp_circle (center 0 0) (end 2.2 0) (layer Cmts.User) (width 0.15))
     (fp_text user %R (at 0.3 0) (layer F.Fab) hide
       (effects (font (size 1 1) (thickness 0.15)))
@@
     (pad "" np_thru_hole circle (at 0 0) (size 2.2 2.2) (drill 2.2) (layers *.Cu *.Mask))
   )
-  (dimension 20 (width 0.15) (layer F.Fab)
-    (gr_text "20.000 mm" (at 346.58125 30 90) (layer F.Fab)
+  (dimension 19.4 (width 0.15) (layer F.Fab)
+    (gr_text "19.400 mm" (at 345.58125 30 90) (layer F.Fab)
       (effects (font (size 1 1) (thickness 0.15)))
     )
-    (feature1 (pts (xy 339.75 20) (xy 345.867671 20)))
-    (feature2 (pts (xy 339.75 40) (xy 345.867671 40)))
-    (crossbar (pts (xy 345.28125 40) (xy 345.28125 20)))
-    (arrow1a (pts (xy 345.28125 20) (xy 345.867671 21.126504)))
-    (arrow1b (pts (xy 345.28125 20) (xy 344.694829 21.126504)))
-    (arrow2a (pts (xy 345.28125 40) (xy 345.867671 38.873496)))
-    (arrow2b (pts (xy 345.28125 40) (xy 344.694829 38.873496)))
+    (feature1 (pts (xy 338.75 20.3) (xy 344.867671 20.3)))
+    (feature2 (pts (xy 338.75 39.7) (xy 344.867671 39.7)))
+    (crossbar (pts (xy 344.28125 39.7) (xy 344.28125 20.3)))
+    (arrow1a (pts (xy 344.28125 20.3) (xy 344.867671 21.426504)))
+    (arrow1b (pts (xy 344.28125 20.3) (xy 343.694829 21.426504)))
+    (arrow2a (pts (xy 344.28125 39.7) (xy 344.867671 38.573496)))
+    (arrow2b (pts (xy 344.28125 39.7) (xy 343.694829 38.573496)))
   )
-  (dimension 172.875 (width 0.15) (layer F.Fab)
-    (gr_text "172.875 mm" (at 253.3125 46.54375) (layer F.Fab)
+  (dimension 171.875 (width 0.15) (layer F.Fab)
+    (gr_text "171.875 mm" (at 252.8125 46.24375) (layer F.Fab)
       (effects (font (size 1 1) (thickness 0.15)))
     )
-    (feature1 (pts (xy 166.875 40) (xy 166.875 45.830171)))
-    (feature2 (pts (xy 339.75 40) (xy 339.75 45.830171)))
-    (crossbar (pts (xy 339.75 45.24375) (xy 166.875 45.24375)))
-    (arrow1a (pts (xy 166.875 45.24375) (xy 168.001504 44.657329)))
-    (arrow1b (pts (xy 166.875 45.24375) (xy 168.001504 45.830171)))
-    (arrow2a (pts (xy 339.75 45.24375) (xy 338.623496 44.657329)))
-    (arrow2b (pts (xy 339.75 45.24375) (xy 338.623496 45.830171)))
+    (feature1 (pts (xy 166.875 39.7) (xy 166.875 45.530171)))
+    (feature2 (pts (xy 338.75 39.7) (xy 338.75 45.530171)))
+    (crossbar (pts (xy 338.75 44.94375) (xy 166.875 44.94375)))
+    (arrow1a (pts (xy 166.875 44.94375) (xy 168.001504 44.357329)))
+    (arrow1b (pts (xy 166.875 44.94375) (xy 168.001504 45.530171)))
+    (arrow2a (pts (xy 338.75 44.94375) (xy 337.623496 44.357329)))
+    (arrow2b (pts (xy 338.75 44.94375) (xy 337.623496 45.530171)))
   )
-  (gr_line (start 186.875 20.3) (end 339.75 20.3) (layer Edge.Cuts) (width 0.1))
+  (gr_line (start 186.875 20.3) (end 338.75 20.3) (layer Edge.Cuts) (width 0.1))
   (gr_line (start 172.875 33) (end 172.875 30) (layer Edge.Cuts) (width 0.1))
   (gr_arc (start 169.875 33) (end 169.875 36) (angle -90) (layer Edge.Cuts) (width 0.1))
@@
   (gr_line (start 172.875 30) (end 183.875 30) (layer Edge.Cuts) (width 0.1))
   (gr_line (start 166.875 39.7) (end 166.875 36) (layer Edge.Cuts) (width 0.1))
-  (gr_line (start 339.75 39.7) (end 339.75 20.3) (layer Edge.Cuts) (width 0.1))
-  (gr_line (start 166.875 39.7) (end 339.75 39.7) (layer Edge.Cuts) (width 0.1))
+  (gr_line (start 338.75 39.7) (end 338.75 20.3) (layer Edge.Cuts) (width 0.1))
+  (gr_line (start 166.875 39.7) (end 338.75 39.7) (layer Edge.Cuts) (width 0.1))
   (zone (net 0) (net_name "") (layer F.Cu) (hatch edge 0.508)
     (connect_pads (clearance 0.508))

Commit message: ケース修正に伴う修正
Other:
- board size 171.9 x 19.4 mm -> 171.4 x 19.4 mm
Changed lines of the file:
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@@
       (effects (font (size 1 1) (thickness 0.15)))
     )
+    (fp_circle (center 0 0) (end 2.45 0) (layer F.CrtYd) (width 0.05))
     (fp_circle (center 0 0) (end 2.2 0) (layer Cmts.User) (width 0.15))
-    (fp_circle (center 0 0) (end 2.45 0) (layer F.CrtYd) (width 0.05))
     (fp_text user %R (at 0.3 0) (layer F.Fab) hide
       (effects (font (size 1 1) (thickness 0.15)))
@@
       (effects (font (size 1 1) (thickness 0.15)))
     )
+    (fp_circle (center 0 0) (end 2.45 0) (layer F.CrtYd) (width 0.05))
     (fp_circle (center 0 0) (end 2.2 0) (layer Cmts.User) (width 0.15))
-    (fp_circle (center 0 0) (end 2.45 0) (layer F.CrtYd) (width 0.05))
     (fp_text user %R (at 0.3 0) (layer F.Fab) hide
       (effects (font (size 1 1) (thickness 0.15)))
@@
       (effects (font (size 1 1) (thickness 0.15)))
     )
+    (fp_circle (center 0 0) (end 2.45 0) (layer F.CrtYd) (width 0.05))
     (fp_circle (center 0 0) (end 2.2 0) (layer Cmts.User) (width 0.15))
-    (fp_circle (center 0 0) (end 2.45 0) (layer F.CrtYd) (width 0.05))
     (fp_text user %R (at 0.3 0) (layer F.Fab) hide
       (effects (font (size 1 1) (thickness 0.15)))
@@
   )
   (dimension 19.4 (width 0.15) (layer F.Fab)
-    (gr_text "19.400 mm" (at 345.58125 30 90) (layer F.Fab)
+    (gr_text "19.400 mm" (at 345.08625 30.005 90) (layer F.Fab)
       (effects (font (size 1 1) (thickness 0.15)))
     )
-    (feature1 (pts (xy 338.75 20.3) (xy 344.867671 20.3)))
-    (feature2 (pts (xy 338.75 39.7) (xy 344.867671 39.7)))
-    (crossbar (pts (xy 344.28125 39.7) (xy 344.28125 20.3)))
-    (arrow1a (pts (xy 344.28125 20.3) (xy 344.867671 21.426504)))
-    (arrow1b (pts (xy 344.28125 20.3) (xy 343.694829 21.426504)))
-    (arrow2a (pts (xy 344.28125 39.7) (xy 344.867671 38.573496)))
-    (arrow2b (pts (xy 344.28125 39.7) (xy 343.694829 38.573496)))
+    (feature1 (pts (xy 338.255 20.305) (xy 344.372671 20.305)))
+    (feature2 (pts (xy 338.255 39.705) (xy 344.372671 39.705)))
+    (crossbar (pts (xy 343.78625 39.705) (xy 343.78625 20.305)))
+    (arrow1a (pts (xy 343.78625 20.305) (xy 344.372671 21.431504)))
+    (arrow1b (pts (xy 343.78625 20.305) (xy 343.199829 21.431504)))
+    (arrow2a (pts (xy 343.78625 39.705) (xy 344.372671 38.578496)))
+    (arrow2b (pts (xy 343.78625 39.705) (xy 343.199829 38.578496)))
   )
-  (dimension 171.875 (width 0.15) (layer F.Fab)
-    (gr_text "171.875 mm" (at 252.8125 46.24375) (layer F.Fab)
+  (dimension 171.38 (width 0.15) (layer F.Fab)
+    (gr_text "171.380 mm" (at 252.564809 46.24625 -0.001671600522) (layer F.Fab)
       (effects (font (size 1 1) (thickness 0.15)))
     )
-    (feature1 (pts (xy 166.875 39.7) (xy 166.875 45.530171)))
-    (feature2 (pts (xy 338.75 39.7) (xy 338.75 45.530171)))
-    (crossbar (pts (xy 338.75 44.94375) (xy 166.875 44.94375)))
-    (arrow1a (pts (xy 166.875 44.94375) (xy 168.001504 44.357329)))
-    (arrow1b (pts (xy 166.875 44.94375) (xy 168.001504 45.530171)))
-    (arrow2a (pts (xy 338.75 44.94375) (xy 337.623496 44.357329)))
-    (arrow2b (pts (xy 338.75 44.94375) (xy 337.623496 45.530171)))
+    (feature1 (pts (xy 166.875 39.7) (xy 166.87483 45.530171)))
+    (feature2 (pts (xy 338.255 39.705) (xy 338.25483 45.535171)))
+    (crossbar (pts (xy 338.254847 44.94875) (xy 166.874847 44.94375)))
+    (arrow1a (pts (xy 166.874847 44.94375) (xy 168.001368 44.357362)))
+    (arrow1b (pts (xy 166.874847 44.94375) (xy 168.001334 45.530204)))
+    (arrow2a (pts (xy 338.254847 44.94875) (xy 337.12836 44.362296)))
+    (arrow2b (pts (xy 338.254847 44.94875) (xy 337.128326 45.535138)))
   )
-  (gr_line (start 186.875 20.3) (end 338.75 20.3) (layer Edge.Cuts) (width 0.1))
+  (gr_line (start 186.875 20.3) (end 338.25 20.3) (layer Edge.Cuts) (width 0.1))
   (gr_line (start 172.875 33) (end 172.875 30) (layer Edge.Cuts) (width 0.1))
   (gr_arc (start 169.875 33) (end 169.875 36) (angle -90) (layer Edge.Cuts) (width 0.1))
@@
   (gr_line (start 172.875 30) (end 183.875 30) (layer Edge.Cuts) (width 0.1))
   (gr_line (start 166.875 39.7) (end 166.875 36) (layer Edge.Cuts) (width 0.1))
-  (gr_line (start 338.75 39.7) (end 338.75 20.3) (layer Edge.Cuts) (width 0.1))
-  (gr_line (start 166.875 39.7) (end 338.75 39.7) (layer Edge.Cuts) (width 0.1))
+  (gr_line (start 338.25 39.7) (end 338.25 20.3) (layer Edge.Cuts) (width 0.1))
+  (gr_line (start 166.875 39.7) (end 338.25 39.7) (layer Edge.Cuts) (width 0.1))
   (zone (net 0) (net_name "") (layer F.Cu) (hatch edge 0.508)
     (connect_pads (clearance 0.508))
