File: Parts/BackPlate/Type-C_Connector/65Type-C_Connector.kicad_pcb (KiCad board)
At the start: 2 copper layers, 172.9 x 20 mm, 3 parts

Commit message: 寸法更新とか
Other:
- board size 172.9 x 20 mm -> 172.9 x 19.4 mm
Changed lines of the file:
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@@
     (arrow2b (pts (xy 315.125 20) (xy 315.711421 21.126504)))
   )
-  (gr_line (start 311.75 40) (end 311.75 20) (layer Edge.Cuts) (width 0.1))
-  (gr_arc (start 277.68125 32.68125) (end 277.68125 34.18125) (angle -180) (layer Edge.Cuts) (width 0.1))
-  (gr_line (start 311.75 40) (end 138.875 40) (layer Edge.Cuts) (width 0.1))
+  (gr_line (start 311.75 39.7) (end 311.75 20.3) (layer Edge.Cuts) (width 0.1))
+  (gr_arc (start 278.68125 32.68125) (end 278.68125 34.18125) (angle -180) (layer Edge.Cuts) (width 0.1))
+  (gr_line (start 311.75 39.7) (end 138.875 39.7) (layer Edge.Cuts) (width 0.1))
   (gr_line (start 289.68125 30.93125) (end 283.67125 30.93125) (layer Edge.Cuts) (width 0.1))
-  (gr_line (start 158.875 20) (end 158.875 27) (layer Edge.Cuts) (width 0.1))
-  (gr_arc (start 296.18125 32.68125) (end 296.18125 34.18125) (angle -180) (layer Edge.Cuts) (width 0.1))
+  (gr_line (start 158.875 20.3) (end 158.875 27) (layer Edge.Cuts) (width 0.1))
+  (gr_arc (start 297.18125 32.68125) (end 297.18125 34.18125) (angle -180) (layer Edge.Cuts) (width 0.1))
   (gr_line (start 283.67125 34.43125) (end 289.68125 34.43125) (layer Edge.Cuts) (width 0.1))
   (gr_arc (start 155.875 27) (end 155.875 30) (angle -90) (layer Edge.Cuts) (width 0.1))
-  (gr_line (start 295.671251 31.181251) (end 296.18125 31.18125) (layer Edge.Cuts) (width 0.1))
+  (gr_line (start 294.671251 31.181251) (end 297.18125 31.18125) (layer Edge.Cuts) (width 0.1))
   (gr_arc (start 283.67125 32.68125) (end 283.67125 30.93125) (angle -180) (layer Edge.Cuts) (width 0.1))
   (gr_arc (start 289.68125 32.68125) (end 289.68125 34.43125) (angle -180) (layer Edge.Cuts) (width 0.1))
-  (gr_arc (start 277.18125 32.68125) (end 277.18125 31.18125) (angle -180) (layer Edge.Cuts) (width 0.1))
-  (gr_line (start 296.18125 34.18125) (end 295.681249 34.181282) (layer Edge.Cuts) (width 0.1))
-  (gr_line (start 138.875 33) (end 138.875 40) (layer Edge.Cuts) (width 0.1))
-  (gr_line (start 277.68125 31.18125) (end 277.18125 31.18125) (layer Edge.Cuts) (width 0.1))
-  (gr_line (start 311.75 20) (end 158.875 20) (layer Edge.Cuts) (width 0.1))
+  (gr_arc (start 276.18125 32.68125) (end 276.18125 31.18125) (angle -180) (layer Edge.Cuts) (width 0.1))
+  (gr_line (start 297.18125 34.18125) (end 294.681249 34.181282) (layer Edge.Cuts) (width 0.1))
+  (gr_line (start 138.875 33) (end 138.875 39.7) (layer Edge.Cuts) (width 0.1))
+  (gr_line (start 278.68125 31.18125) (end 276.18125 31.18125) (layer Edge.Cuts) (width 0.1))
+  (gr_line (start 311.75 20.3) (end 158.875 20.3) (layer Edge.Cuts) (width 0.1))
   (gr_line (start 155.875 30) (end 141.875 30) (layer Edge.Cuts) (width 0.1))
   (gr_arc (start 141.875 33) (end 141.875 30) (angle -90) (layer Edge.Cuts) (width 0.1))
-  (gr_line (start 277.68125 34.18125) (end 277.18125 34.18125) (layer Edge.Cuts) (width 0.1))
-  (gr_arc (start 295.68125 32.68125) (end 295.671251 31.181251) (angle -179.6180338) (layer Edge.Cuts) (width 0.1))
+  (gr_line (start 278.68125 34.18125) (end 276.18125 34.18125) (layer Edge.Cuts) (width 0.1))
+  (gr_arc (start 294.68125 32.68125) (end 294.671251 31.181251) (angle -179.6180338) (layer Edge.Cuts) (width 0.1))
   (zone (net 0) (net_name "") (layer F.Cu) (hatch edge 0.508)
     (connect_pads (clearance 0.508))

Commit message: 諸々修正
今度はちゃんと説明書きを書く
Other:
- board size 172.9 x 19.4 mm -> 171.9 x 19.4 mm
Changed lines of the file:
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@@
-(kicad_pcb (version 20171130) (host pcbnew "(5.1.5)-3")
+(kicad_pcb (version 20171130) (host pcbnew "(5.1.10)-1")
   (general
     (thickness 1.6)
@@
     (pad_drill 0)
     (pad_to_mask_clearance 0)
-    (solder_mask_min_width 0.25)
     (aux_axis_origin 47.625 47.625)
     (grid_origin 47.625 47.625)
@@
       (effects (font (size 1 1) (thickness 0.15)))
     )
+    (fp_circle (center 0 0) (end 2.2 0) (layer Cmts.User) (width 0.15))
     (fp_circle (center 0 0) (end 2.45 0) (layer F.CrtYd) (width 0.05))
-    (fp_circle (center 0 0) (end 2.2 0) (layer Cmts.User) (width 0.15))
     (fp_text user %R (at 0.3 0) (layer F.Fab) hide
       (effects (font (size 1 1) (thickness 0.15)))
@@
       (effects (font (size 1 1) (thickness 0.15)))
     )
+    (fp_circle (center 0 0) (end 2.2 0) (layer Cmts.User) (width 0.15))
     (fp_circle (center 0 0) (end 2.45 0) (layer F.CrtYd) (width 0.05))
-    (fp_circle (center 0 0) (end 2.2 0) (layer Cmts.User) (width 0.15))
     (fp_text user %R (at 0.3 0) (layer F.Fab) hide
       (effects (font (size 1 1) (thickness 0.15)))
@@
       (effects (font (size 1 1) (thickness 0.15)))
     )
+    (fp_circle (center 0 0) (end 2.2 0) (layer Cmts.User) (width 0.15))
     (fp_circle (center 0 0) (end 2.45 0) (layer F.CrtYd) (width 0.05))
-    (fp_circle (center 0 0) (end 2.2 0) (layer Cmts.User) (width 0.15))
     (fp_text user %R (at 0.3 0) (layer F.Fab) hide
       (effects (font (size 1 1) (thickness 0.15)))
@@
     (pad "" np_thru_hole circle (at 0 0 180) (size 2.2 2.2) (drill 2.2) (layers *.Cu *.Mask))
   )
-  (dimension 172.875 (width 0.15) (layer F.Fab)
-    (gr_text "172.875 mm" (at 225.3125 45.625) (layer F.Fab)
+  (dimension 171.875 (width 0.15) (layer F.Fab)
+    (gr_text "171.875 mm" (at 224.8125 45.325) (layer F.Fab)
       (effects (font (size 1 1) (thickness 0.15)))
     )
-    (feature1 (pts (xy 138.875 40) (xy 138.875 44.911421)))
-    (feature2 (pts (xy 311.75 40) (xy 311.75 44.911421)))
-    (crossbar (pts (xy 311.75 44.325) (xy 138.875 44.325)))
-    (arrow1a (pts (xy 138.875 44.325) (xy 140.001504 43.738579)))
-    (arrow1b (pts (xy 138.875 44.325) (xy 140.001504 44.911421)))
-    (arrow2a (pts (xy 311.75 44.325) (xy 310.623496 43.738579)))
-    (arrow2b (pts (xy 311.75 44.325) (xy 310.623496 44.911421)))
+    (feature1 (pts (xy 138.875 39.7) (xy 138.875 44.611421)))
+    (feature2 (pts (xy 310.75 39.7) (xy 310.75 44.611421)))
+    (crossbar (pts (xy 310.75 44.025) (xy 138.875 44.025)))
+    (arrow1a (pts (xy 138.875 44.025) (xy 140.001504 43.438579)))
+    (arrow1b (pts (xy 138.875 44.025) (xy 140.001504 44.611421)))
+    (arrow2a (pts (xy 310.75 44.025) (xy 309.623496 43.438579)))
+    (arrow2b (pts (xy 310.75 44.025) (xy 309.623496 44.611421)))
   )
-  (dimension 20 (width 0.15) (layer F.Fab)
-    (gr_text "20.000 mm" (at 316.425 30 270) (layer F.Fab)
+  (dimension 19.4 (width 0.15) (layer F.Fab)
+    (gr_text "19.400 mm" (at 315.425 30 270) (layer F.Fab)
       (effects (font (size 1 1) (thickness 0.15)))
     )
-    (feature1 (pts (xy 311.75 40) (xy 315.711421 40)))
-    (feature2 (pts (xy 311.75 20) (xy 315.711421 20)))
-    (crossbar (pts (xy 315.125 20) (xy 315.125 40)))
-    (arrow1a (pts (xy 315.125 40) (xy 314.538579 38.873496)))
-    (arrow1b (pts (xy 315.125 40) (xy 315.711421 38.873496)))
-    (arrow2a (pts (xy 315.125 20) (xy 314.538579 21.126504)))
-    (arrow2b (pts (xy 315.125 20) (xy 315.711421 21.126504)))
+    (feature1 (pts (xy 310.75 39.7) (xy 314.711421 39.7)))
+    (feature2 (pts (xy 310.75 20.3) (xy 314.711421 20.3)))
+    (crossbar (pts (xy 314.125 20.3) (xy 314.125 39.7)))
+    (arrow1a (pts (xy 314.125 39.7) (xy 313.538579 38.573496)))
+    (arrow1b (pts (xy 314.125 39.7) (xy 314.711421 38.573496)))
+    (arrow2a (pts (xy 314.125 20.3) (xy 313.538579 21.426504)))
+    (arrow2b (pts (xy 314.125 20.3) (xy 314.711421 21.426504)))
   )
-  (gr_line (start 311.75 39.7) (end 311.75 20.3) (layer Edge.Cuts) (width 0.1))
+  (gr_line (start 310.75 39.7) (end 310.75 20.3) (layer Edge.Cuts) (width 0.1))
   (gr_arc (start 278.68125 32.68125) (end 278.68125 34.18125) (angle -180) (layer Edge.Cuts) (width 0.1))
-  (gr_line (start 311.75 39.7) (end 138.875 39.7) (layer Edge.Cuts) (width 0.1))
+  (gr_line (start 310.75 39.7) (end 138.875 39.7) (layer Edge.Cuts) (width 0.1))
   (gr_line (start 289.68125 30.93125) (end 283.67125 30.93125) (layer Edge.Cuts) (width 0.1))
   (gr_line (start 158.875 20.3) (end 158.875 27) (layer Edge.Cuts) (width 0.1))
@@
   (gr_line (start 138.875 33) (end 138.875 39.7) (layer Edge.Cuts) (width 0.1))
   (gr_line (start 278.68125 31.18125) (end 276.18125 31.18125) (layer Edge.Cuts) (width 0.1))
-  (gr_line (start 311.75 20.3) (end 158.875 20.3) (layer Edge.Cuts) (width 0.1))
+  (gr_line (start 310.75 20.3) (end 158.875 20.3) (layer Edge.Cuts) (width 0.1))
   (gr_line (start 155.875 30) (end 141.875 30) (layer Edge.Cuts) (width 0.1))
   (gr_arc (start 141.875 33) (end 141.875 30) (angle -90) (layer Edge.Cuts) (width 0.1))

Commit message: ケース修正に伴う修正
Other:
- board size 171.9 x 19.4 mm -> 171.4 x 19.4 mm
Changed lines of the file:
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@@
       (effects (font (size 1 1) (thickness 0.15)))
     )
+    (fp_circle (center 0 0) (end 2.45 0) (layer F.CrtYd) (width 0.05))
     (fp_circle (center 0 0) (end 2.2 0) (layer Cmts.User) (width 0.15))
-    (fp_circle (center 0 0) (end 2.45 0) (layer F.CrtYd) (width 0.05))
     (fp_text user %R (at 0.3 0) (layer F.Fab) hide
       (effects (font (size 1 1) (thickness 0.15)))
@@
       (effects (font (size 1 1) (thickness 0.15)))
     )
+    (fp_circle (center 0 0) (end 2.45 0) (layer F.CrtYd) (width 0.05))
     (fp_circle (center 0 0) (end 2.2 0) (layer Cmts.User) (width 0.15))
-    (fp_circle (center 0 0) (end 2.45 0) (layer F.CrtYd) (width 0.05))
     (fp_text user %R (at 0.3 0) (layer F.Fab) hide
       (effects (font (size 1 1) (thickness 0.15)))
@@
       (effects (font (size 1 1) (thickness 0.15)))
     )
+    (fp_circle (center 0 0) (end 2.45 0) (layer F.CrtYd) (width 0.05))
     (fp_circle (center 0 0) (end 2.2 0) (layer Cmts.User) (width 0.15))
-    (fp_circle (center 0 0) (end 2.45 0) (layer F.CrtYd) (width 0.05))
     (fp_text user %R (at 0.3 0) (layer F.Fab) hide
       (effects (font (size 1 1) (thickness 0.15)))
@@
     (pad "" np_thru_hole circle (at 0 0 180) (size 2.2 2.2) (drill 2.2) (layers *.Cu *.Mask))
   )
-  (dimension 171.875 (width 0.15) (layer F.Fab)
-    (gr_text "171.875 mm" (at 224.8125 45.325) (layer F.Fab)
+  (dimension 171.375 (width 0.15) (layer F.Fab)
+    (gr_text "171.375 mm" (at 224.5625 45.325) (layer F.Fab)
       (effects (font (size 1 1) (thickness 0.15)))
     )
     (feature1 (pts (xy 138.875 39.7) (xy 138.875 44.611421)))
-    (feature2 (pts (xy 310.75 39.7) (xy 310.75 44.611421)))
-    (crossbar (pts (xy 310.75 44.025) (xy 138.875 44.025)))
+    (feature2 (pts (xy 310.25 39.7) (xy 310.25 44.611421)))
+    (crossbar (pts (xy 310.25 44.025) (xy 138.875 44.025)))
     (arrow1a (pts (xy 138.875 44.025) (xy 140.001504 43.438579)))
     (arrow1b (pts (xy 138.875 44.025) (xy 140.001504 44.611421)))
-    (arrow2a (pts (xy 310.75 44.025) (xy 309.623496 43.438579)))
-    (arrow2b (pts (xy 310.75 44.025) (xy 309.623496 44.611421)))
+    (arrow2a (pts (xy 310.25 44.025) (xy 309.123496 43.438579)))
+    (arrow2b (pts (xy 310.25 44.025) (xy 309.123496 44.611421)))
   )
   (dimension 19.4 (width 0.15) (layer F.Fab)
-    (gr_text "19.400 mm" (at 315.425 30 270) (layer F.Fab)
+    (gr_text "19.400 mm" (at 314.925 30 270) (layer F.Fab)
       (effects (font (size 1 1) (thickness 0.15)))
     )
-    (feature1 (pts (xy 310.75 39.7) (xy 314.711421 39.7)))
-    (feature2 (pts (xy 310.75 20.3) (xy 314.711421 20.3)))
-    (crossbar (pts (xy 314.125 20.3) (xy 314.125 39.7)))
-    (arrow1a (pts (xy 314.125 39.7) (xy 313.538579 38.573496)))
-    (arrow1b (pts (xy 314.125 39.7) (xy 314.711421 38.573496)))
-    (arrow2a (pts (xy 314.125 20.3) (xy 313.538579 21.426504)))
-    (arrow2b (pts (xy 314.125 20.3) (xy 314.711421 21.426504)))
+    (feature1 (pts (xy 310.25 39.7) (xy 314.211421 39.7)))
+    (feature2 (pts (xy 310.25 20.3) (xy 314.211421 20.3)))
+    (crossbar (pts (xy 313.625 20.3) (xy 313.625 39.7)))
+    (arrow1a (pts (xy 313.625 39.7) (xy 313.038579 38.573496)))
+    (arrow1b (pts (xy 313.625 39.7) (xy 314.211421 38.573496)))
+    (arrow2a (pts (xy 313.625 20.3) (xy 313.038579 21.426504)))
+    (arrow2b (pts (xy 313.625 20.3) (xy 314.211421 21.426504)))
   )
-  (gr_line (start 310.75 39.7) (end 310.75 20.3) (layer Edge.Cuts) (width 0.1))
+  (gr_line (start 310.25 39.7) (end 310.25 20.3) (layer Edge.Cuts) (width 0.1))
   (gr_arc (start 278.68125 32.68125) (end 278.68125 34.18125) (angle -180) (layer Edge.Cuts) (width 0.1))
-  (gr_line (start 310.75 39.7) (end 138.875 39.7) (layer Edge.Cuts) (width 0.1))
+  (gr_line (start 310.25 39.7) (end 138.875 39.7) (layer Edge.Cuts) (width 0.1))
   (gr_line (start 289.68125 30.93125) (end 283.67125 30.93125) (layer Edge.Cuts) (width 0.1))
   (gr_line (start 158.875 20.3) (end 158.875 27) (layer Edge.Cuts) (width 0.1))
@@
   (gr_line (start 138.875 33) (end 138.875 39.7) (layer Edge.Cuts) (width 0.1))
   (gr_line (start 278.68125 31.18125) (end 276.18125 31.18125) (layer Edge.Cuts) (width 0.1))
-  (gr_line (start 310.75 20.3) (end 158.875 20.3) (layer Edge.Cuts) (width 0.1))
+  (gr_line (start 310.25 20.3) (end 158.875 20.3) (layer Edge.Cuts) (width 0.1))
   (gr_line (start 155.875 30) (end 141.875 30) (layer Edge.Cuts) (width 0.1))
   (gr_arc (start 141.875 33) (end 141.875 30) (angle -90) (layer Edge.Cuts) (width 0.1))
