File: Parts/BackPlate/kbd67/kbd67Back.kicad_pcb (KiCad board)
At the start: 2 copper layers, 172.9 x 20 mm, 3 parts

Commit message: 寸法更新とか
Other:
- board size 172.9 x 20 mm -> 172.9 x 19.4 mm
Changed lines of the file:
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@@
   (gr_line (start 279.3 23.2) (end 285.3 23.2) (layer Edge.Cuts) (width 0.1))
   (gr_line (start 285.3 32.2) (end 279.3 32.2) (layer Edge.Cuts) (width 0.1))
-  (gr_line (start 311.8 20) (end 158.925 20) (layer Edge.Cuts) (width 0.1))
-  (gr_line (start 311.8 40) (end 138.925 40) (layer Edge.Cuts) (width 0.1))
+  (gr_line (start 311.8 20.3) (end 158.925 20.3) (layer Edge.Cuts) (width 0.1))
+  (gr_line (start 311.8 39.7) (end 138.925 39.7) (layer Edge.Cuts) (width 0.1))
   (gr_arc (start 141.925 33) (end 141.925 30) (angle -90) (layer Edge.Cuts) (width 0.1))
   (gr_arc (start 155.925 27) (end 155.925 30) (angle -90) (layer Edge.Cuts) (width 0.1))
-  (gr_line (start 138.925 33) (end 138.925 40) (layer Edge.Cuts) (width 0.1))
+  (gr_line (start 138.925 33) (end 138.925 39.7) (layer Edge.Cuts) (width 0.1))
   (gr_line (start 155.925 30) (end 141.925 30) (layer Edge.Cuts) (width 0.1))
-  (gr_line (start 158.925 20) (end 158.925 27) (layer Edge.Cuts) (width 0.1))
-  (gr_line (start 311.8 40) (end 311.8 20) (layer Edge.Cuts) (width 0.1))
+  (gr_line (start 158.925 20.3) (end 158.925 27) (layer Edge.Cuts) (width 0.1))
+  (gr_line (start 311.8 39.7) (end 311.8 20.3) (layer Edge.Cuts) (width 0.1))
   (zone (net 0) (net_name "") (layer F.Cu) (hatch edge 0.508)
     (connect_pads (clearance 0.508))

Commit message: 諸々修正
今度はちゃんと説明書きを書く
Other:
- board size 172.9 x 19.4 mm -> 171.9 x 19.4 mm
Changed lines of the file:
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@@
-(kicad_pcb (version 20171130) (host pcbnew "(5.1.5)-3")
+(kicad_pcb (version 20171130) (host pcbnew "(5.1.10)-1")
   (general
     (thickness 1.6)
@@
     (pad_drill 0)
     (pad_to_mask_clearance 0)
-    (solder_mask_min_width 0.25)
     (aux_axis_origin 47.625 47.625)
     (grid_origin 47.625 47.625)
@@
       (effects (font (size 1 1) (thickness 0.15)))
     )
+    (fp_circle (center 0 0) (end 2.2 0) (layer Cmts.User) (width 0.15))
     (fp_circle (center 0 0) (end 2.45 0) (layer F.CrtYd) (width 0.05))
-    (fp_circle (center 0 0) (end 2.2 0) (layer Cmts.User) (width 0.15))
     (fp_text user %R (at 0.3 0) (layer F.Fab) hide
       (effects (font (size 1 1) (thickness 0.15)))
@@
       (effects (font (size 1 1) (thickness 0.15)))
     )
+    (fp_circle (center 0 0) (end 2.2 0) (layer Cmts.User) (width 0.15))
     (fp_circle (center 0 0) (end 2.45 0) (layer F.CrtYd) (width 0.05))
-    (fp_circle (center 0 0) (end 2.2 0) (layer Cmts.User) (width 0.15))
     (fp_text user %R (at 0.3 0) (layer F.Fab) hide
       (effects (font (size 1 1) (thickness 0.15)))
@@
       (effects (font (size 1 1) (thickness 0.15)))
     )
+    (fp_circle (center 0 0) (end 2.2 0) (layer Cmts.User) (width 0.15))
     (fp_circle (center 0 0) (end 2.45 0) (layer F.CrtYd) (width 0.05))
-    (fp_circle (center 0 0) (end 2.2 0) (layer Cmts.User) (width 0.15))
     (fp_text user %R (at 0.3 0) (layer F.Fab) hide
       (effects (font (size 1 1) (thickness 0.15)))
@@
     (pad "" np_thru_hole circle (at 0 0 180) (size 2.2 2.2) (drill 2.2) (layers *.Cu *.Mask))
   )
-  (dimension 20 (width 0.15) (layer F.Fab)
-    (gr_text "20.000 mm" (at 316.225 30 270) (layer F.Fab)
+  (dimension 19.4 (width 0.15) (layer F.Fab)
+    (gr_text "19.400 mm" (at 315.225 30 270) (layer F.Fab)
       (effects (font (size 1 1) (thickness 0.15)))
     )
-    (feature1 (pts (xy 311.8 40) (xy 315.511421 40)))
-    (feature2 (pts (xy 311.8 20) (xy 315.511421 20)))
-    (crossbar (pts (xy 314.925 20) (xy 314.925 40)))
-    (arrow1a (pts (xy 314.925 40) (xy 314.338579 38.873496)))
-    (arrow1b (pts (xy 314.925 40) (xy 315.511421 38.873496)))
-    (arrow2a (pts (xy 314.925 20) (xy 314.338579 21.126504)))
-    (arrow2b (pts (xy 314.925 20) (xy 315.511421 21.126504)))
+    (feature1 (pts (xy 310.8 39.7) (xy 314.511421 39.7)))
+    (feature2 (pts (xy 310.8 20.3) (xy 314.511421 20.3)))
+    (crossbar (pts (xy 313.925 20.3) (xy 313.925 39.7)))
+    (arrow1a (pts (xy 313.925 39.7) (xy 313.338579 38.573496)))
+    (arrow1b (pts (xy 313.925 39.7) (xy 314.511421 38.573496)))
+    (arrow2a (pts (xy 313.925 20.3) (xy 313.338579 21.426504)))
+    (arrow2b (pts (xy 313.925 20.3) (xy 314.511421 21.426504)))
   )
-  (dimension 172.875 (width 0.15) (layer F.Fab)
-    (gr_text "172.875 mm" (at 225.3625 44.1625) (layer F.Fab)
+  (dimension 171.875 (width 0.15) (layer F.Fab)
+    (gr_text "171.875 mm" (at 224.8625 43.8625) (layer F.Fab)
       (effects (font (size 1 1) (thickness 0.15)))
     )
-    (feature1 (pts (xy 138.925 40) (xy 138.925 43.448921)))
-    (feature2 (pts (xy 311.8 40) (xy 311.8 43.448921)))
-    (crossbar (pts (xy 311.8 42.8625) (xy 138.925 42.8625)))
-    (arrow1a (pts (xy 138.925 42.8625) (xy 140.051504 42.276079)))
-    (arrow1b (pts (xy 138.925 42.8625) (xy 140.051504 43.448921)))
-    (arrow2a (pts (xy 311.8 42.8625) (xy 310.673496 42.276079)))
-    (arrow2b (pts (xy 311.8 42.8625) (xy 310.673496 43.448921)))
+    (feature1 (pts (xy 138.925 39.7) (xy 138.925 43.148921)))
+    (feature2 (pts (xy 310.8 39.7) (xy 310.8 43.148921)))
+    (crossbar (pts (xy 310.8 42.5625) (xy 138.925 42.5625)))
+    (arrow1a (pts (xy 138.925 42.5625) (xy 140.051504 41.976079)))
+    (arrow1b (pts (xy 138.925 42.5625) (xy 140.051504 43.148921)))
+    (arrow2a (pts (xy 310.8 42.5625) (xy 309.673496 41.976079)))
+    (arrow2b (pts (xy 310.8 42.5625) (xy 309.673496 43.148921)))
   )
   (gr_text KBD67mk2 (at 253 35.5) (layer B.Cu)
@@
   (gr_line (start 279.3 23.2) (end 285.3 23.2) (layer Edge.Cuts) (width 0.1))
   (gr_line (start 285.3 32.2) (end 279.3 32.2) (layer Edge.Cuts) (width 0.1))
-  (gr_line (start 311.8 20.3) (end 158.925 20.3) (layer Edge.Cuts) (width 0.1))
-  (gr_line (start 311.8 39.7) (end 138.925 39.7) (layer Edge.Cuts) (width 0.1))
+  (gr_line (start 310.8 20.3) (end 158.925 20.3) (layer Edge.Cuts) (width 0.1))
+  (gr_line (start 310.8 39.7) (end 138.925 39.7) (layer Edge.Cuts) (width 0.1))
   (gr_arc (start 141.925 33) (end 141.925 30) (angle -90) (layer Edge.Cuts) (width 0.1))
   (gr_arc (start 155.925 27) (end 155.925 30) (angle -90) (layer Edge.Cuts) (width 0.1))
@@
   (gr_line (start 155.925 30) (end 141.925 30) (layer Edge.Cuts) (width 0.1))
   (gr_line (start 158.925 20.3) (end 158.925 27) (layer Edge.Cuts) (width 0.1))
-  (gr_line (start 311.8 39.7) (end 311.8 20.3) (layer Edge.Cuts) (width 0.1))
+  (gr_line (start 310.8 39.7) (end 310.8 20.3) (layer Edge.Cuts) (width 0.1))
   (zone (net 0) (net_name "") (layer F.Cu) (hatch edge 0.508)
     (connect_pads (clearance 0.508))

Commit message: ケース修正に伴う修正
Other:
- board size 171.9 x 19.4 mm -> 171.4 x 19.4 mm
Changed lines of the file:
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@@
       (effects (font (size 1 1) (thickness 0.15)))
     )
+    (fp_circle (center 0 0) (end 2.45 0) (layer F.CrtYd) (width 0.05))
     (fp_circle (center 0 0) (end 2.2 0) (layer Cmts.User) (width 0.15))
-    (fp_circle (center 0 0) (end 2.45 0) (layer F.CrtYd) (width 0.05))
     (fp_text user %R (at 0.3 0) (layer F.Fab) hide
       (effects (font (size 1 1) (thickness 0.15)))
@@
       (effects (font (size 1 1) (thickness 0.15)))
     )
+    (fp_circle (center 0 0) (end 2.45 0) (layer F.CrtYd) (width 0.05))
     (fp_circle (center 0 0) (end 2.2 0) (layer Cmts.User) (width 0.15))
-    (fp_circle (center 0 0) (end 2.45 0) (layer F.CrtYd) (width 0.05))
     (fp_text user %R (at 0.3 0) (layer F.Fab) hide
       (effects (font (size 1 1) (thickness 0.15)))
@@
       (effects (font (size 1 1) (thickness 0.15)))
     )
+    (fp_circle (center 0 0) (end 2.45 0) (layer F.CrtYd) (width 0.05))
     (fp_circle (center 0 0) (end 2.2 0) (layer Cmts.User) (width 0.15))
-    (fp_circle (center 0 0) (end 2.45 0) (layer F.CrtYd) (width 0.05))
     (fp_text user %R (at 0.3 0) (layer F.Fab) hide
       (effects (font (size 1 1) (thickness 0.15)))
@@
   )
   (dimension 19.4 (width 0.15) (layer F.Fab)
-    (gr_text "19.400 mm" (at 315.225 30 270) (layer F.Fab)
+    (gr_text "19.400 mm" (at 314.725 30 270) (layer F.Fab)
       (effects (font (size 1 1) (thickness 0.15)))
     )
-    (feature1 (pts (xy 310.8 39.7) (xy 314.511421 39.7)))
-    (feature2 (pts (xy 310.8 20.3) (xy 314.511421 20.3)))
-    (crossbar (pts (xy 313.925 20.3) (xy 313.925 39.7)))
-    (arrow1a (pts (xy 313.925 39.7) (xy 313.338579 38.573496)))
-    (arrow1b (pts (xy 313.925 39.7) (xy 314.511421 38.573496)))
-    (arrow2a (pts (xy 313.925 20.3) (xy 313.338579 21.426504)))
-    (arrow2b (pts (xy 313.925 20.3) (xy 314.511421 21.426504)))
+    (feature1 (pts (xy 310.3 39.7) (xy 314.011421 39.7)))
+    (feature2 (pts (xy 310.3 20.3) (xy 314.011421 20.3)))
+    (crossbar (pts (xy 313.425 20.3) (xy 313.425 39.7)))
+    (arrow1a (pts (xy 313.425 39.7) (xy 312.838579 38.573496)))
+    (arrow1b (pts (xy 313.425 39.7) (xy 314.011421 38.573496)))
+    (arrow2a (pts (xy 313.425 20.3) (xy 312.838579 21.426504)))
+    (arrow2b (pts (xy 313.425 20.3) (xy 314.011421 21.426504)))
   )
-  (dimension 171.875 (width 0.15) (layer F.Fab)
-    (gr_text "171.875 mm" (at 224.8625 43.8625) (layer F.Fab)
+  (dimension 171.375 (width 0.15) (layer F.Fab)
+    (gr_text "171.375 mm" (at 224.6125 43.8625) (layer F.Fab)
       (effects (font (size 1 1) (thickness 0.15)))
     )
     (feature1 (pts (xy 138.925 39.7) (xy 138.925 43.148921)))
-    (feature2 (pts (xy 310.8 39.7) (xy 310.8 43.148921)))
-    (crossbar (pts (xy 310.8 42.5625) (xy 138.925 42.5625)))
+    (feature2 (pts (xy 310.3 39.7) (xy 310.3 43.148921)))
+    (crossbar (pts (xy 310.3 42.5625) (xy 138.925 42.5625)))
     (arrow1a (pts (xy 138.925 42.5625) (xy 140.051504 41.976079)))
     (arrow1b (pts (xy 138.925 42.5625) (xy 140.051504 43.148921)))
-    (arrow2a (pts (xy 310.8 42.5625) (xy 309.673496 41.976079)))
-    (arrow2b (pts (xy 310.8 42.5625) (xy 309.673496 43.148921)))
+    (arrow2a (pts (xy 310.3 42.5625) (xy 309.173496 41.976079)))
+    (arrow2b (pts (xy 310.3 42.5625) (xy 309.173496 43.148921)))
   )
   (gr_text KBD67mk2 (at 253 35.5) (layer B.Cu)
@@
   (gr_line (start 279.3 23.2) (end 285.3 23.2) (layer Edge.Cuts) (width 0.1))
   (gr_line (start 285.3 32.2) (end 279.3 32.2) (layer Edge.Cuts) (width 0.1))
-  (gr_line (start 310.8 20.3) (end 158.925 20.3) (layer Edge.Cuts) (width 0.1))
-  (gr_line (start 310.8 39.7) (end 138.925 39.7) (layer Edge.Cuts) (width 0.1))
+  (gr_line (start 310.3 20.3) (end 158.925 20.3) (layer Edge.Cuts) (width 0.1))
+  (gr_line (start 310.3 39.7) (end 138.925 39.7) (layer Edge.Cuts) (width 0.1))
   (gr_arc (start 141.925 33) (end 141.925 30) (angle -90) (layer Edge.Cuts) (width 0.1))
   (gr_arc (start 155.925 27) (end 155.925 30) (angle -90) (layer Edge.Cuts) (width 0.1))
@@
   (gr_line (start 155.925 30) (end 141.925 30) (layer Edge.Cuts) (width 0.1))
   (gr_line (start 158.925 20.3) (end 158.925 27) (layer Edge.Cuts) (width 0.1))
-  (gr_line (start 310.8 39.7) (end 310.8 20.3) (layer Edge.Cuts) (width 0.1))
+  (gr_line (start 310.3 39.7) (end 310.3 20.3) (layer Edge.Cuts) (width 0.1))
   (zone (net 0) (net_name "") (layer F.Cu) (hatch edge 0.508)
     (connect_pads (clearance 0.508))
