File: Keyboard/J73GL/1_Top/J73GL_Top.sch (KiCad schematic (older format))
At the start: 259 parts, among them J1 Conn_01x02, J10 Conn_01x01, J11 Conn_01x01, J12 Conn_01x01, J13 Conn_01x01, J14 Conn_01x01, J15 Conn_01x01, J16 Conn_01x01, J17 Conn_01x01, J2 Conn_01x01, J3 Conn_01x01, J4 Conn_01x01, J5 Conn_01x01, J6 Conn_01x01, J7 Conn_01x01, J8 Conn_01x01, J9 Conn_01x01, SW1 SW_PUSH, SW10 SW_PUSH, SW11 SW_PUSH, SW12 SW_PUSH, SW13 SW_PUSH, SW14 SW_PUSH, SW15 SW_PUSH, SW16 SW_PUSH, SW17 SW_PUSH, SW18 SW_PUSH, SW19 SW_PUSH, SW2 SW_PUSH, SW20 SW_PUSH, SW21 SW_PUSH, SW22 SW_PUSH, SW23 SW_PUSH, SW24 SW_PUSH, SW25 SW_PUSH, SW26 SW_PUSH, SW27 SW_PUSH, SW28 SW_PUSH, SW29 SW_PUSH, SW3 SW_PUSH, SW30 SW_PUSH, SW31 SW_PUSH, SW32 SW_PUSH, SW33 SW_PUSH, SW34 SW_PUSH, SW35 SW_PUSH, SW36 SW_PUSH, SW37 SW_PUSH, SW38 SW_PUSH, SW39 SW_PUSH, SW4 SW_PUSH, SW40 SW_PUSH, SW41 SW_PUSH, SW42 SW_PUSH, SW43 SW_PUSH, SW44 SW_PUSH, SW45 SW_PUSH, SW46 SW_PUSH, SW47 SW_PUSH, SW48 SW_PUSH, SW49 SW_PUSH, SW5 SW_PUSH, SW50 SW_PUSH, SW51 SW_PUSH, SW52 SW_PUSH, SW53 SW_PUSH, SW54 SW_PUSH, SW55 SW_PUSH, SW56 SW_PUSH, SW57 SW_PUSH, SW58 SW_PUSH, SW59 SW_PUSH, SW6 SW_PUSH, SW60 SW_PUSH, SW61 SW_PUSH, SW62 SW_PUSH, SW63 SW_PUSH, SW64 SW_PUSH, SW65 SW_PUSH, SW66 SW_PUSH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

Commit message: 諸々修正
今度はちゃんと説明書きを書く
Other:
- note added: "The grid size should be set to 25mils."
Changed lines of the file:
@@
 $EndComp
 $Comp
-L power:GND #PWR025
-U 1 1 5CC518DD
-P 15250 9075
-F 0 "#PWR025" H 15250 8825 50  0001 C CNN
-F 1 "GND" H 15255 8902 50  0000 C CNN
-F 2 "" H 15250 9075 50  0001 C CNN
-F 3 "" H 15250 9075 50  0001 C CNN
-	1    15250 9075
-	1    0    0    -1
-$EndComp
-$Comp
 L Connector_Generic:Conn_01x01 J15
 U 1 1 5CC9EE7D
@@
 	10175 12425 10175 13075
 NoConn ~ 9925 13275
+Text Notes 5850 900  0    50   ~ 0
+The grid size should be set to 25mils.
+$Comp
+L power:GND #PWR?
+U 1 1 61BB629E
+P 15250 9075
+F 0 "#PWR?" H 15250 8825 50  0001 C CNN
+F 1 "GND" H 15255 8902 50  0000 C CNN
+F 2 "" H 15250 9075 50  0001 C CNN
+F 3 "" H 15250 9075 50  0001 C CNN
+	1    15250 9075
+	1    0    0    -1
+$EndComp
 $EndSCHEMATC

Commit message: バックアップファイルの整理
Parts:
- U1: symbol kbd:BLEMicroPro -> Salicylic_kbd:Micon_BLEMicroPro
Changed lines of the file:
@@
 BLE Micro Pro
 $Comp
-L kbd:BLEMicroPro U1
+L Salicylic_kbd:Micon_BLEMicroPro U1
 U 1 1 5BF16C54
 P 2150 1975

Commit message: シンボル、フットプリントの更新に合わせて更新
Parts:
- removed L11, L12, L13, L14, L15, L16, L17, L18, L19, L20, L21, L22, L23, L24, L25, L26, L27, L28, L29, L30, L31, L32, L33, L34, L35, L36, L37, L38, L39, L40, L41, L42, L43, L44, L45, L46, L47, L48, L49, L50, L51, L52, L53, L54, L55, L56, L57, L58, L59, L60, L61, L62, L63, L64, L65, L66, L67, L68, L69, L70, L71, L72, L73, L74, L75, L76, L77, L78, L79, L80: SK6812MINI, kbd_Parts:LED_SK6812MINI-E_BL, symbol kbd:SK6812MINI
- added L11, L12, L13, L14, L15, L16, L17, L18, L19, L20, L21, L22, L23, L24, L25, L26, L27, L28, L29, L30, L31, L32, L33, L34, L35, L36, L37, L38, L39, L40, L41, L42, L43, L44, L45, L46, L47, L48, L49, L50, L51, L52, L53, L54, L55, L56, L57, L58, L59, L60, L61, L62, L63, L64, L65, L66, L67, L68, L69, L70, L71, L72, L73, L74, L75, L76, L77, L78, L79, L80: SK6812MINI, kbd_Parts:LED_SK6812MINI-E_BL, symbol Salicylic_kbd:LED_SK6812MINI-E
- L1, L10, L2, L3, L4, L5, L6, L7, L8, L9: symbol kbd:SK6812MINI -> Salicylic_kbd:LED_SK6812MINI-E
- SW1, SW10, SW11, SW12, SW13, SW14, SW15, SW16, SW17, SW18, SW19, SW2, SW20, SW21, SW22, SW23, SW24, SW25, SW26, SW27, SW28, SW29, SW3, SW30, SW31, SW32, SW33, SW34, SW35, SW36, SW37, SW38, SW39, SW4, SW40, SW41, SW42, SW43, SW44, SW45, SW46, SW47, SW48, SW49, SW5, SW50, SW51, SW52, SW53, SW54, SW55, SW56, SW57, SW58, SW59, SW6, SW60, SW61, SW62, SW63, SW64, SW65, SW66, SW67, SW68, SW69, SW7, SW70, SW71, SW72, SW73, SW74, SW75, SW76, SW77, SW78, SW79, SW8, SW80, SW81, SW9: symbol kbd:SW_PUSH -> Switch:SW_Push
Connections:
- wire segments 913 -> 349
Other:
- note removed: "The grid size should be set to 25mils."
- moved on the sheet: D1, D10, D11, D12, D13, D14, D15, D16, D17, D18, D19, D2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
