File: Keyboard/J73GL/1_Top/J73GL_Top.kicad_pcb (KiCad board)
At the start: 2 copper layers, 315.4 x 99.2 mm, 89 parts, among them J10 Conn_01x01, J11 Conn_01x01, J12 Conn_01x01, J13 Conn_01x01, J14 Conn_01x01, J15 Conn_01x01, J16 Conn_01x01, J17 Conn_01x01, J2 Conn_01x01, J3 Conn_01x01, J4 Conn_01x01, J5 Conn_01x01, J6 Conn_01x01, J7 Conn_01x01, J8 Conn_01x01, J9 Conn_01x01, SW1 SW_PUSH, SW2 KEY_SWITCH, SW3 SW_PUSH, SW4 KEY_SWITCH, SW4 SW_PUSH, SW5 SW_PUSH, SW7 SW_PUSH, SW8 SW_PUSH

Commit message: 寸法更新とか
Other:
- board size 315.4 x 99.2 mm -> 314.4 x 98.8 mm
Changed lines of the file:
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@@
   (gr_line (start 78.575 20.55) (end 264.325 20.55) (layer F.Fab) (width 0.15))
   (gr_line (start 10.45 50.55) (end 332.4 50.55) (layer F.Fab) (width 0.15))
-  (gr_arc (start 320.825 20.05) (end 323.825 20.05) (angle -90) (layer F.Fab) (width 0.1))
-  (gr_arc (start 320.825 113.25) (end 320.825 116.25) (angle -90) (layer F.Fab) (width 0.1))
-  (gr_arc (start 22.075 20.05) (end 22.075 17.05) (angle -90) (layer F.Fab) (width 0.1))
-  (gr_arc (start 22.075 113.25) (end 19.075 113.25) (angle -90) (layer F.Fab) (width 0.1))
+  (gr_arc (start 320.625 20.25) (end 323.625 20.25) (angle -90) (layer F.Fab) (width 0.1))
+  (gr_arc (start 320.625 113.05) (end 320.625 116.05) (angle -90) (layer F.Fab) (width 0.1))
+  (gr_arc (start 22.275 20.25) (end 22.275 17.25) (angle -90) (layer F.Fab) (width 0.1))
+  (gr_arc (start 22.275 113.05) (end 19.275 113.05) (angle -90) (layer F.Fab) (width 0.1))
   (gr_text "Do not place switches to the left of this line." (at 32.5 13.7) (layer F.Fab)
     (effects (font (size 1 1) (thickness 0.15)))
@@
     (effects (font (size 1 1) (thickness 0.15)))
   )
-  (gr_line (start 323.825 20.05) (end 323.825 113.25) (layer F.Fab) (width 0.1))
-  (gr_line (start 19.075 20.05) (end 19.075 113.25) (layer F.Fab) (width 0.1))
-  (gr_arc (start 16.775 113.25) (end 13.775 113.25) (angle -90) (layer Edge.Cuts) (width 0.1))
-  (gr_arc (start 16.775 20.05) (end 16.775 17.05) (angle -90) (layer Edge.Cuts) (width 0.1))
-  (gr_arc (start 326.125 20.05) (end 329.125 20.05) (angle -90) (layer Edge.Cuts) (width 0.1))
-  (gr_arc (start 326.125 113.25) (end 326.125 116.25) (angle -90) (layer Edge.Cuts) (width 0.1))
-  (gr_line (start 329.125 113.25) (end 329.125 20.05) (layer Edge.Cuts) (width 0.1))
-  (gr_line (start 16.775 116.25) (end 326.125 116.25) (layer Edge.Cuts) (width 0.1))
-  (gr_line (start 13.775 20.05) (end 13.775 113.25) (layer Edge.Cuts) (width 0.1))
-  (gr_line (start 326.125 17.05) (end 16.775 17.05) (layer Edge.Cuts) (width 0.1))
+  (gr_line (start 323.625 20.25) (end 323.625 113.05) (layer F.Fab) (width 0.1))
+  (gr_line (start 19.275 20.25) (end 19.275 113.05) (layer F.Fab) (width 0.1))
+  (gr_arc (start 17.275 113.05) (end 14.275 113.05) (angle -90) (layer Edge.Cuts) (width 0.1))
+  (gr_arc (start 17.275 20.25) (end 17.275 17.25) (angle -90) (layer Edge.Cuts) (width 0.1))
+  (gr_arc (start 325.625 20.25) (end 328.625 20.25) (angle -90) (layer Edge.Cuts) (width 0.1))
+  (gr_arc (start 325.625 113.05) (end 325.625 116.05) (angle -90) (layer Edge.Cuts) (width 0.1))
+  (gr_line (start 328.625 113.05) (end 328.625 20.25) (layer Edge.Cuts) (width 0.1))
+  (gr_line (start 17.275 116.05) (end 325.625 116.05) (layer Edge.Cuts) (width 0.1))
+  (gr_line (start 14.275 20.25) (end 14.275 113.05) (layer Edge.Cuts) (width 0.1))
+  (gr_line (start 325.625 17.25) (end 17.275 17.25) (layer Edge.Cuts) (width 0.1))
 )

Commit message: スイッチ穴の寸法を14.1mmに変更
Parts:
- SW1, SW4 (x28), SW7, SW8 (x32): footprint kbd_SW_Hole:SW_Hole -> kbd_SW_Hole:SW_Hole_1

Commit message: フットプリント名の変更に対応
Parts:
- SW1, SW4 (x28), SW7, SW8 (x32): footprint kbd_SW_Hole:SW_Hole_1 -> kbd_SW_Hole:SW_Hole_1u
- SW2: footprint kbd_SW_Hole:SW_Hole_1.5 -> kbd_SW_Hole:SW_Hole_1.5u
- SW3, SW8: footprint kbd_SW_Hole:SW_Hole_1.75 -> kbd_SW_Hole:SW_Hole_1.75u
- SW4: footprint kbd_SW_Hole:SW_Hole_2 -> kbd_SW_Hole:SW_Hole_2u
- SW4: footprint kbd_SW_Hole:SW_Hole_2.25 -> kbd_SW_Hole:SW_Hole_2.25u
- SW5 (x4), SW7 (x2): footprint kbd_SW_Hole:SW_Hole_1.25 -> kbd_SW_Hole:SW_Hole_1.25u
