File: Keyboard/J73GL/3_Decoration/J73GL_Decoration.sch (KiCad schematic (older format))
At the start: 259 parts, among them J1 Conn_01x02, J10 Conn_01x01, J11 Conn_01x01, J12 Conn_01x01, J13 Conn_01x01, J14 Conn_01x01, J15 Conn_01x01, J16 Conn_01x01, J17 Conn_01x01, J2 Conn_01x01, J3 Conn_01x01, J4 Conn_01x01, J5 Conn_01x01, J6 Conn_01x01, J7 Conn_01x01, J8 Conn_01x01, J9 Conn_01x01, SW1 SW_PUSH, SW10 SW_PUSH, SW11 SW_PUSH, SW12 SW_PUSH, SW13 SW_PUSH, SW14 SW_PUSH, SW15 SW_PUSH, SW16 SW_PUSH, SW17 SW_PUSH, SW18 SW_PUSH, SW19 SW_PUSH, SW2 SW_PUSH, SW20 SW_PUSH, SW21 SW_PUSH, SW22 SW_PUSH, SW23 SW_PUSH, SW24 SW_PUSH, SW25 SW_PUSH, SW26 SW_PUSH, SW27 SW_PUSH, SW28 SW_PUSH, SW29 SW_PUSH, SW3 SW_PUSH, SW30 SW_PUSH, SW31 SW_PUSH, SW32 SW_PUSH, SW33 SW_PUSH, SW34 SW_PUSH, SW35 SW_PUSH, SW36 SW_PUSH, SW37 SW_PUSH, SW38 SW_PUSH, SW39 SW_PUSH, SW4 SW_PUSH, SW40 SW_PUSH, SW41 SW_PUSH, SW42 SW_PUSH, SW43 SW_PUSH, SW44 SW_PUSH, SW45 SW_PUSH, SW46 SW_PUSH, SW47 SW_PUSH, SW48 SW_PUSH, SW49 SW_PUSH, SW5 SW_PUSH, SW50 SW_PUSH, SW51 SW_PUSH, SW52 SW_PUSH, SW53 SW_PUSH, SW54 SW_PUSH, SW55 SW_PUSH, SW56 SW_PUSH, SW57 SW_PUSH, SW58 SW_PUSH, SW59 SW_PUSH, SW6 SW_PUSH, SW60 SW_PUSH, SW61 SW_PUSH, SW62 SW_PUSH, SW63 SW_PUSH, SW64 SW_PUSH, SW65 SW_PUSH, SW66 SW_PUSH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

Commit message: バックアップファイルの整理
Parts:
- U1: symbol kbd:BLEMicroPro -> Salicylic_kbd:Micon_BLEMicroPro
Changed lines of the file:
@@
 BLE Micro Pro
 $Comp
-L kbd:BLEMicroPro U1
+L Salicylic_kbd:Micon_BLEMicroPro U1
 U 1 1 5BF16C54
 P 2150 1975

Commit message: シンボル、フットプリントの更新に合わせて更新
Parts:
- removed L10, L11, L12, L14, L15, L16, L18, L19, L2, L20, L22, L23, L24, L26, L27, L28, L3, L30, L31, L32, L34, L35, L36, L38, L39, L4, L40, L41, L42, L43, L44, L45, L46, L47, L48, L49, L50, L51, L52, L53, L54, L55, L56, L57, L58, L59, L6, L60, L61, L62, L63, L64, L65, L66, L67, L68, L69, L7, L70, L71, L72, L73, L74, L75, L76, L77, L78, L79, L8, L80: SK6812MINI, kbd:YS-SK6812MINI-E_v3, symbol kbd:SK6812MINI
- added L11, L12, L13, L14, L15, L16, L17, L18, L19, L20, L21, L22, L23, L24, L25, L26, L27, L28, L29, L30, L31, L32, L33, L34, L35, L36, L37, L38, L39, L40, L41, L42, L43, L44, L45, L46, L47, L48, L49, L50, L51, L52, L53, L54, L55, L56, L57, L58, L59, L60, L61, L62, L63, L64, L65, L66, L67, L68, L69, L70, L71, L72, L73, L74, L75, L76, L77, L78, L79, L80: SK6812MINI, kbd_Parts:LED_SK6812MINI-E_BL, symbol Salicylic_kbd:LED_SK6812MINI-E
- D1, D10, D11, D12, D13, D14, D15, D16, D17, D18, D19, D2, D20, D21, D22, D23, D24, D25, D26, D27, D28, D29, D3, D30, D31, D32, D33, D34, D35, D36, D37, D38, D39, D4, D40, D41, D42, D43, D44, D45, D46, D47, D48, D49, D5, D50, D51, D52, D53, D54, D55, D56, D57, D58, D59, D6, D60, D61, D62, D63, D64, D65, D66, D67, D68, D69, D7, D70, D71, D72, D73, D74, D75, D76, D77, D78, D79, D8, D80, D9: footprint kbd:D3_TH_SMD_BL -> kbd_Parts:Diode_TH_SMD
- J1: footprint kbd:XH2.5_rev -> kbd_Parts:Battery_XH2.5_GL
- J10, J11, J12, J13, J14, J15, J16, J17, J8, J9: footprint kbd:HOLE_m2_Outline_Fab -> kbd_Hole:m2_Screw_Hole_Fab
- J2, J3, J4, J5, J6, J7: footprint kbd:HOLE_m2_Outline -> kbd_Hole:m2_Screw_Hole_EdgeCuts
- L1: footprint kbd:YS-SK6812MINI-E_v3 -> kbd_Parts:LED_SK6812MINI-E_BL; symbol kbd:SK6812MINI -> Salicylic_kbd:LED_SK6812MINI-E
- L10: renamed from L37; footprint kbd:YS-SK6812MINI-E_v3 -> kbd_Parts:LED_SK6812MINI-E_BL; symbol kbd:SK6812MINI -> Salicylic_kbd:LED_SK6812MINI-E
- L2: renamed from L5; footprint kbd:YS-SK6812MINI-E_v3 -> kbd_Parts:LED_SK6812MINI-E_BL; symbol kbd:SK6812MINI -> Salicylic_kbd:LED_SK6812MINI-E
- L3: renamed from L9; footprint kbd:YS-SK6812MINI-E_v3 -> kbd_Parts:LED_SK6812MINI-E_BL; symbol kbd:SK6812MINI -> Salicylic_kbd:LED_SK6812MINI-E
- L4: renamed from L13; footprint kbd:YS-SK6812MINI-E_v3 -> kbd_Parts:LED_SK6812MINI-E_BL; symbol kbd:SK6812MINI -> Salicylic_kbd:LED_SK6812MINI-E
- L5: renamed from L17; footprint kbd:YS-SK6812MINI-E_v3 -> kbd_Parts:LED_SK6812MINI-E_BL; symbol kbd:SK6812MINI -> Salicylic_kbd:LED_SK6812MINI-E
- L6: renamed from L21; footprint kbd:YS-SK6812MINI-E_v3 -> kbd_Parts:LED_SK6812MINI-E_BL; symbol kbd:SK6812MINI -> Salicylic_kbd:LED_SK6812MINI-E
- L7: renamed from L25; footprint kbd:YS-SK6812MINI-E_v3 -> kbd_Parts:LED_SK6812MINI-E_BL; symbol kbd:SK6812MINI -> Salicylic_kbd:LED_SK6812MINI-E
- L8: renamed from L29; footprint kbd:YS-SK6812MINI-E_v3 -> kbd_Parts:LED_SK6812MINI-E_BL; symbol kbd:SK6812MINI -> Salicylic_kbd:LED_SK6812MINI-E
- L9: renamed from L33; footprint kbd:YS-SK6812MINI-E_v3 -> kbd_Parts:LED_SK6812MINI-E_BL; symbol kbd:SK6812MINI -> Salicylic_kbd:LED_SK6812MINI-E
- SW1, SW10, SW11, SW12, SW13, SW14, SW15, SW16, SW17, SW18, SW19, SW2, SW20, SW21, SW22, SW23, SW24, SW25, SW26, SW27, SW28, SW29, SW3, SW30, SW31, SW32, SW33, SW34, SW35, SW36, SW37, SW38, SW39, SW4, SW40, SW41, SW42, SW43, SW44, SW45, SW46, SW47, SW48, SW49, SW5, SW50, SW51, SW52, SW53, SW54, SW55, SW56, SW57, SW58, SW59, SW6, SW60, SW61, SW62, SW63, SW64, SW65, SW66, SW67, SW68, SW69, SW7, SW70, SW71, SW72, SW73, SW74, SW75, SW76, SW77, SW78, SW79, SW8, SW80, SW9: footprint kbd:CherryMX_Choc_Hotswap_LH_v2 -> kbd_SW:CherryMX_Choc_Hotswap_1u; symbol kbd:SW_PUSH -> Switch:SW_Push
- SW81: footprint kbd:ResetSW -> kbd_Parts:ResetSW; symbol kbd:SW_PUSH -> Switch:SW_Push
- U1: footprint kbd:BLE_Micro_Pro_L1 -> kbd_Parts:Micon_BMP_GL
Connections:
- wire segments 906 -> 349
Other:
- note added: "Left hand block (Max 40 keys)"
- note added: "Right hand block (Max 40 keys)"
- note removed: "Left hand block (Max 35 keys)"
- note removed: "Right hand block (Max 35 keys)"
- moved on the sheet: D1, D10, D11, D12, D13, D14, D15, D16, D17, D18, D19, D2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
