File: Keyboard/A52GL/2_Assemble/A52GL_Assemble.sch (KiCad schematic (older format))
At the start: 123 parts, among them J1 Conn_01x02, J10 Conn_01x01, J11 Conn_01x01, J12 Conn_01x01, J13 Conn_01x01, J14 Conn_01x01, J15 Conn_01x01, J16 Conn_01x01, J17 Conn_01x01, J2 Conn_01x01, J3 Conn_01x01, J4 Conn_01x01, J5 Conn_01x01, J6 Conn_01x01, J7 Conn_01x01, J8 Conn_01x01, J9 Conn_01x01, SW1 SW_PUSH, SW10 SW_PUSH, SW11 SW_PUSH, SW12 SW_PUSH, SW13 SW_PUSH, SW14 SW_PUSH, SW15 SW_PUSH, SW16 SW_PUSH, SW17 SW_PUSH, SW18 SW_PUSH, SW19 SW_PUSH, SW2 SW_PUSH, SW20 SW_PUSH, SW21 SW_PUSH, SW22 SW_PUSH, SW23 SW_PUSH, SW24 SW_PUSH, SW25 SW_PUSH, SW26 SW_PUSH, SW27 SW_PUSH, SW28 SW_PUSH, SW29 SW_PUSH, SW3 SW_PUSH, SW30 SW_PUSH, SW31 SW_PUSH, SW32 SW_PUSH, SW33 SW_PUSH, SW34 SW_PUSH, SW35 SW_PUSH, SW36 SW_PUSH, SW37 SW_PUSH, SW38 SW_PUSH, SW39 SW_PUSH, SW4 SW_PUSH, SW40 SW_PUSH, SW41 SW_PUSH, SW42 SW_PUSH, SW43 SW_PUSH, SW44 SW_PUSH, SW45 SW_PUSH, SW46 SW_PUSH, SW47 SW_PUSH, SW48 SW_PUSH, SW49 SW_PUSH, SW5 SW_PUSH, SW50 SW_PUSH, SW51 SW_PUSH, SW52 SW_PUSH, SW53 SW_PUSH, SW6 SW_PUSH, SW7 SW_PUSH, SW8 SW_PUSH, SW9 SW_PUSH, U1 BLEMicroPro

Commit message: バックアップファイルの整理
Parts:
- U1: symbol kbd:BLEMicroPro -> Salicylic_kbd:Micon_BLEMicroPro
Changed lines of the file:
@@
 BLE Micro Pro
 $Comp
-L kbd:BLEMicroPro U1
+L Salicylic_kbd:Micon_BLEMicroPro U1
 U 1 1 5BF16C54
 P 2150 1975

Commit message: シンボル、フットプリントの更新に合わせて更新
Parts:
- D1, D10, D11, D12, D13, D14, D15, D16, D17, D18, D19, D2, D20, D21, D22, D23, D24, D25, D26, D27, D28, D29, D3, D30, D31, D32, D33, D34, D35, D36, D37, D38, D39, D4, D40, D41, D42, D43, D44, D45, D46, D47, D48, D49, D5, D50, D51, D52, D6, D7, D8, D9: footprint kbd:D3_TH_SMD_BL -> kbd_Parts:Diode_TH_SMD
- J1: footprint kbd:XH2.5_rev -> kbd_Parts:Battery_XH2.5_GL_PCB
- J10, J11, J12, J13, J14, J15, J16, J17, J8, J9: footprint kbd:HOLE_m2_Outline_Fab -> kbd_Hole:m2_Screw_Hole_Fab
- J2, J3, J4, J5, J6, J7: footprint kbd:HOLE_m2_Outline -> kbd_Hole:m2_Screw_Hole_EdgeCuts
- SW1, SW10, SW11, SW12, SW13, SW14, SW15, SW16, SW17, SW18, SW20, SW21, SW22, SW23, SW24, SW25, SW26, SW28, SW29, SW30, SW31, SW32, SW33, SW35, SW36, SW37, SW38, SW39, SW40, SW41, SW42, SW43, SW44, SW45, SW46, SW48, SW49, SW5, SW51, SW52, SW6, SW7, SW9: footprint kbd:CherryMX_Hotswap_BL_LH_v2 -> kbd_SW:CherryMX_Hotswap_1.0u; symbol kbd:SW_PUSH -> Switch:SW_Push
- SW19: footprint kbd:CherryMX_Hotswap_2u_BL_2 -> kbd_SW:CherryMX_Hotswap_2u; symbol kbd:SW_PUSH -> Switch:SW_Push
- SW2, SW34, SW4, SW8: footprint kbd:CherryMX_Hotswap_1.25u_LH_v2 -> kbd_SW:CherryMX_Hotswap_1.25u; symbol kbd:SW_PUSH -> Switch:SW_Push
- SW27, SW47: footprint kbd:CherryMX_Hotswap_2.25u_BL_v2 -> kbd_SW:CherryMX_Hotswap_2.25u; symbol kbd:SW_PUSH -> Switch:SW_Push
- SW3: footprint kbd:CherryMX_Hotswap_1.75u_BL_LH_v2 -> kbd_SW:CherryMX_Hotswap_1.75u; symbol kbd:SW_PUSH -> Switch:SW_Push
- SW50: footprint kbd:CherryMX_Hotswap_BL_LH_v2_ -> kbd_SW:CherryMX_Hotswap_1.0u_Small1; symbol kbd:SW_PUSH -> Switch:SW_Push
- SW53: footprint kbd:ResetSW -> kbd_Parts:ResetSW; symbol kbd:SW_PUSH -> Switch:SW_Push
- U1: footprint kbd:BLE_Micro_Pro_L1 -> kbd_Parts:Micon_BMP_GL
Other:
- moved on the sheet: D1, D10, D11, D12, D13, D14, D15, D16, D17, D18, D19, D2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

Commit message: フットプリント名の変更に対応
Parts:
- SW1, SW10, SW11, SW12, SW13, SW14, SW15, SW16, SW17, SW18, SW20, SW21, SW22, SW23, SW24, SW25, SW26, SW28, SW29, SW30, SW31, SW32, SW33, SW35, SW36, SW37, SW38, SW39, SW40, SW41, SW42, SW43, SW44, SW45, SW46, SW48, SW49, SW5, SW51, SW52, SW6, SW7, SW9: footprint kbd_SW:CherryMX_Hotswap_1.0u -> kbd_SW:CherryMX_Hotswap_1u
- SW50: footprint kbd_SW:CherryMX_Hotswap_1.0u_Small1 -> kbd_SW:CherryMX_Hotswap_1u_Small1
