File: Keyboard/A52GL/2_Assemble_PCBA/A52GL_Assemble.kicad_pcb (KiCad board)
At the start: 2 copper layers, 304.4 x 116.9 mm, 115 parts, among them J1 Conn_01x02, SW1 SW_PUSH, SW10 SW_PUSH, SW11 SW_PUSH, SW12 SW_PUSH, SW13 SW_PUSH, SW14 SW_PUSH, SW15 SW_PUSH, SW16 SW_PUSH, SW17 SW_PUSH, SW18 SW_PUSH, SW19 SW_PUSH, SW2 SW_PUSH, SW20 SW_PUSH, SW21 SW_PUSH, SW22 SW_PUSH, SW23 SW_PUSH, SW24 SW_PUSH, SW25 SW_PUSH, SW26 SW_PUSH, SW27 SW_PUSH, SW28 SW_PUSH, SW29 SW_PUSH, SW3 SW_PUSH, SW30 SW_PUSH, SW31 SW_PUSH, SW32 SW_PUSH, SW33 SW_PUSH, SW34 SW_PUSH, SW35 SW_PUSH, SW36 SW_PUSH, SW37 SW_PUSH, SW38 SW_PUSH, SW39 SW_PUSH, SW4 SW_PUSH, SW40 SW_PUSH, SW41 SW_PUSH, SW42 SW_PUSH, SW43 SW_PUSH, SW44 SW_PUSH, SW45 SW_PUSH, SW46 SW_PUSH, SW47 SW_PUSH, SW48 SW_PUSH, SW49 SW_PUSH, SW5 SW_PUSH, SW50 SW_PUSH, SW51 SW_PUSH, SW52 SW_PUSH, SW53 SW_PUSH, SW6 SW_PUSH, SW7 SW_PUSH, SW8 SW_PUSH, SW9 SW_PUSH, U1 BLEMicroPro

Commit message: シンボル、フットプリントの更新に合わせて更新
Parts:
- SW50: footprint kbd:CherryMX_Hotswap_BL_LH_v2_ -> kbd_SW:CherryMX_Hotswap_1.0u_Small1

Commit message: フットプリント名の変更に対応
Parts:
- SW1, SW10, SW11, SW12, SW13, SW14, SW15, SW16, SW17, SW18, SW20, SW21, SW22, SW23, SW24, SW25, SW26, SW28, SW29, SW30, SW31, SW32, SW33, SW35, SW36, SW37, SW38, SW39, SW40, SW41, SW42, SW43, SW44, SW45, SW46, SW48, SW49, SW5, SW51, SW52, SW6, SW7, SW9: footprint kbd_SW:CherryMX_Hotswap_1.0u -> kbd_SW:CherryMX_Hotswap_1u
- SW50: footprint kbd_SW:CherryMX_Hotswap_1.0u_Small1 -> kbd_SW:CherryMX_Hotswap_1u_Small1
