File: Keyboard/J73GL/1_Top_TH/J73GL_Top.kicad_pcb (KiCad board)
At the start: 2 copper layers, 315.4 x 99.2 mm, 89 parts, among them J10 Conn_01x01, J11 Conn_01x01, J12 Conn_01x01, J13 Conn_01x01, J14 Conn_01x01, J15 Conn_01x01, J16 Conn_01x01, J17 Conn_01x01, J2 Conn_01x01, J3 Conn_01x01, J4 Conn_01x01, J5 Conn_01x01, J6 Conn_01x01, J7 Conn_01x01, J8 Conn_01x01, J9 Conn_01x01, SW1 SW_PUSH, SW2 KEY_SWITCH, SW3 SW_PUSH, SW4 KEY_SWITCH, SW4 SW_PUSH, SW5 SW_PUSH, SW7 SW_PUSH, SW8 SW_PUSH

Commit message: 寸法更新とか
Other:
- board size 315.4 x 99.2 mm -> 314.4 x 98.8 mm

Commit message: フットプリント名の変更に対応
Parts:
- SW1, SW4 (x28), SW7, SW8 (x32): footprint kbd_SW_Hole:SW_Hole_TH -> kbd_SW_Hole:SW_Hole_TH_1u
- SW2: footprint kbd_SW_Hole:SW_Hole_TH_1.5 -> kbd_SW_Hole:SW_Hole_TH_1.5u
- SW3, SW8: footprint kbd_SW_Hole:SW_Hole_TH_1.75 -> kbd_SW_Hole:SW_Hole_TH_1.75u
- SW4: footprint kbd_SW_Hole:SW_Hole_TH_2 -> kbd_SW_Hole:SW_Hole_TH_2u
- SW4: footprint kbd_SW_Hole:SW_Hole_TH_2.25 -> kbd_SW_Hole:SW_Hole_TH_2.25u
- SW5 (x4), SW7 (x2): footprint kbd_SW_Hole:SW_Hole_TH_1.25 -> kbd_SW_Hole:SW_Hole_TH_1.25u
