File: Keyboard/N51GL/1_Top/Naked51_Top.kicad_pcb (KiCad board)
At the start: 2 copper layers, 315.8 x 99.2 mm, 58 parts, among them SW10 SW_PUSH, SW11 SW_PUSH, SW13 SW_PUSH, SW14 SW_PUSH, SW15 SW_PUSH, SW16 SW_PUSH, SW18 SW_PUSH, SW19 SW_PUSH, SW2 KEY_SWITCH, SW20 SW_PUSH, SW23 SW_PUSH, SW24 SW_PUSH, SW25 SW_PUSH, SW27 SW_PUSH, SW28 SW_PUSH, SW29 SW_PUSH, SW30 SW_PUSH, SW32 SW_PUSH, SW33 SW_PUSH, SW34 SW_PUSH, SW35 SW_PUSH, SW37 SW_PUSH, SW38 SW_PUSH, SW39 SW_PUSH, SW4 SW_PUSH, SW40 SW_PUSH, SW42 SW_PUSH, SW43 SW_PUSH, SW44 SW_PUSH, SW46 SW_PUSH, SW47 SW_PUSH, SW48 SW_PUSH, SW49 SW_PUSH, SW5 SW_PUSH, SW51 SW_PUSH, SW52 SW_PUSH, SW53 SW_PUSH, SW54 SW_PUSH, SW56 SW_PUSH, SW57 SW_PUSH, SW58 SW_PUSH, SW59 SW_PUSH, SW6 SW_PUSH, SW61 SW_PUSH, SW62 SW_PUSH, SW63 SW_PUSH, SW64 SW_PUSH, SW7 SW_PUSH, SW9 SW_PUSH

Commit message: 寸法更新とか
Parts:
- moved Ref** 0.50 mm to (16.1, 111.8)
- moved Ref** 0.50 mm to (16.1, 21.6)
- moved Ref** 0.50 mm to (326.8, 111.8)
- moved Ref** 0.50 mm to (326.8, 21.6)
Other:
- board size 315.8 x 99.2 mm -> 314.4 x 98.8 mm
Changed lines of the file:
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@@
   (general
     (thickness 1.6)
-    (drawings 55)
+    (drawings 57)
     (tracks 1)
     (zones 0)
@@
   )
   (module kbd:HOLE_m2_a (layer F.Cu)
-    (at 16.075 111.25)
+    (at 16.075 111.75)
     (descr "Mounting Hole 2.2mm, no annular, M2")
     (tags "mounting hole 2.2mm no annular m2")
@@
   )
   (module kbd:HOLE_m2_a (layer F.Cu)
-    (at 16.075 66.7)
+    (at 16.075 66.65)
     (descr "Mounting Hole 2.2mm, no annular, M2")
     (tags "mounting hole 2.2mm no annular m2")
@@
   )
   (module kbd:HOLE_m2_a (layer F.Cu)
-    (at 16.075 22.05)
+    (at 16.075 21.55)
     (descr "Mounting Hole 2.2mm, no annular, M2")
     (tags "mounting hole 2.2mm no annular m2")
@@
   )
   (module kbd:HOLE_m2_a (layer F.Cu)
-    (at 326.825 111.25)
+    (at 326.825 111.75)
     (descr "Mounting Hole 2.2mm, no annular, M2")
     (tags "mounting hole 2.2mm no annular m2")
@@
   )
   (module kbd:HOLE_m2_a (layer F.Cu)
-    (at 326.825 66.7)
+    (at 326.825 66.65)
     (descr "Mounting Hole 2.2mm, no annular, M2")
     (tags "mounting hole 2.2mm no annular m2")
@@
   )
   (module kbd:HOLE_m2_a (layer F.Cu)
-    (at 326.825 22.05)
+    (at 326.825 21.55)
     (descr "Mounting Hole 2.2mm, no annular, M2")
     (tags "mounting hole 2.2mm no annular m2")
@@
     )
   )
+  (gr_line (start 13.575 19.55) (end 13.575 113.75) (layer F.Fab) (width 0.15))
+  (gr_line (start 329.325 19.55) (end 329.325 113.75) (layer F.Fab) (width 0.15))
   (gr_circle (center 169.008711 85) (end 184.008711 85) (layer F.Fab) (width 0.1))
   (gr_line (start 10.075 122.75) (end 8.575 121.25) (layer F.Fab) (width 0.15))
@@
   (gr_circle (center 234.325 120.25) (end 235.425 120.25) (layer F.Fab) (width 0.1))
   (gr_circle (center 11.075 13.05) (end 12.175 13.05) (layer F.Fab) (width 0.1))
-  (gr_circle (center 11.075 66.7) (end 12.175 66.7) (layer F.Fab) (width 0.1))
+  (gr_circle (center 11.075 66.65) (end 12.175 66.65) (layer F.Fab) (width 0.1))
   (gr_circle (center 11.075 120.25) (end 12.175 120.25) (layer F.Fab) (width 0.1))
   (gr_circle (center 331.825 13.05) (end 332.925 13.05) (layer F.Fab) (width 0.1))
-  (gr_circle (center 331.825 66.7) (end 332.925 66.7) (layer F.Fab) (width 0.1))
+  (gr_circle (center 331.825 66.65) (end 332.925 66.65) (layer F.Fab) (width 0.1))
   (gr_circle (center 331.825 120.25) (end 332.925 120.25) (layer F.Fab) (width 0.1))
   (gr_line (start 10.075 122.75) (end 332.825 122.75) (layer F.Fab) (width 0.15))
@@
   (gr_line (start 78.575 20.55) (end 264.325 20.55) (layer F.Fab) (width 0.15))
   (gr_line (start 10.45 50.55) (end 332.4 50.55) (layer F.Fab) (width 0.15))
-  (gr_arc (start 321.325 20.05) (end 324.325 20.05) (angle -90) (layer F.Fab) (width 0.1))
-  (gr_arc (start 321.325 113.25) (end 321.325 116.25) (angle -90) (layer F.Fab) (width 0.1))
-  (gr_arc (start 21.575 20.05) (end 21.575 17.05) (angle -90) (layer F.Fab) (width 0.1))
-  (gr_arc (start 21.575 113.25) (end 18.575 113.25) (angle -90) (layer F.Fab) (width 0.1))
+  (gr_arc (start 320.625 20.25) (end 323.625 20.25) (angle -90) (layer F.Fab) (width 0.1))
+  (gr_arc (start 320.625 113.05) (end 320.625 116.05) (angle -90) (layer F.Fab) (width 0.1))
+  (gr_arc (start 22.275 20.25) (end 22.275 17.25) (angle -90) (layer F.Fab) (width 0.1))
+  (gr_arc (start 22.275 113.05) (end 19.275 113.05) (angle -90) (layer F.Fab) (width 0.1))
   (gr_text "Do not place switches to the left of this line." (at 32.5 14.7) (layer F.Fab)
     (effects (font (size 1 1) (thickness 0.15)))
@@
     (effects (font (size 1 1) (thickness 0.15)))
   )
-  (gr_line (start 324.325 20.05) (end 324.325 113.25) (layer F.Fab) (width 0.1))
-  (gr_line (start 18.575 20.05) (end 18.575 113.25) (layer F.Fab) (width 0.1))
-  (gr_arc (start 16.575 113.25) (end 13.575 113.25) (angle -90) (layer Edge.Cuts) (width 0.1))
-  (gr_arc (start 16.575 20.05) (end 16.575 17.05) (angle -90) (layer Edge.Cuts) (width 0.1))
-  (gr_arc (start 326.325 20.05) (end 329.325 20.05) (angle -90) (layer Edge.Cuts) (width 0.1))
-  (gr_arc (start 326.325 113.25) (end 326.325 116.25) (angle -90) (layer Edge.Cuts) (width 0.1))
-  (gr_line (start 329.325 113.25) (end 329.325 20.05) (layer Edge.Cuts) (width 0.1))
-  (gr_line (start 16.575 116.25) (end 326.325 116.25) (layer Edge.Cuts) (width 0.1))
-  (gr_line (start 13.575 20.05) (end 13.575 113.25) (layer Edge.Cuts) (width 0.1))
-  (gr_line (start 326.325 17.05) (end 16.575 17.05) (layer Edge.Cuts) (width 0.1))
+  (gr_line (start 323.625 20.25) (end 323.625 113.05) (layer F.Fab) (width 0.1))
+  (gr_line (start 19.275 20.25) (end 19.275 113.05) (layer F.Fab) (width 0.1))
+  (gr_arc (start 17.275 113.05) (end 14.275 113.05) (angle -90) (layer Edge.Cuts) (width 0.1))
+  (gr_arc (start 17.275 20.25) (end 17.275 17.25) (angle -90) (layer Edge.Cuts) (width 0.1))
+  (gr_arc (start 325.625 20.25) (end 328.625 20.25) (angle -90) (layer Edge.Cuts) (width 0.1))
+  (gr_arc (start 325.625 113.05) (end 325.625 116.05) (angle -90) (layer Edge.Cuts) (width 0.1))
+  (gr_line (start 328.625 113.05) (end 328.625 20.25) (layer Edge.Cuts) (width 0.1))
+  (gr_line (start 17.275 116.05) (end 325.625 116.05) (layer Edge.Cuts) (width 0.1))
+  (gr_line (start 14.275 20.25) (end 14.275 113.05) (layer Edge.Cuts) (width 0.1))
+  (gr_line (start 325.625 17.25) (end 17.275 17.25) (layer Edge.Cuts) (width 0.1))
   (segment (start 216.959123 92.362903) (end 216.959123 92.337904) (width 0.25) (layer B.Cu) (net 1))
 )

Commit message: スイッチ穴の寸法を14.1mmに変更
Parts:
- SW10, SW11, SW13, SW14, SW15, SW18, SW19, SW20, SW23, SW24, SW25, SW27, SW28, SW29, SW30, SW32, SW33, SW34 (x2), SW35, SW37, SW38, SW39, SW4 (x2), SW42, SW43, SW44, SW46, SW47, SW48, SW51, SW52, SW53, SW54, SW56, SW57, SW58, SW59, SW61, SW62, SW63, SW64, SW9: footprint kbd_SW_Hole:SW_Hole -> kbd_SW_Hole:SW_Hole_1

Commit message: フットプリント名の変更に対応
Parts:
- SW10, SW11, SW13, SW14, SW15, SW18, SW19, SW20, SW23, SW24, SW25, SW27, SW28, SW29, SW30, SW32, SW33, SW34 (x2), SW35, SW37, SW38, SW39, SW4 (x2), SW42, SW43, SW44, SW46, SW47, SW48, SW51, SW52, SW53, SW54, SW56, SW57, SW58, SW59, SW61, SW62, SW63, SW64, SW9: footprint kbd_SW_Hole:SW_Hole_1 -> kbd_SW_Hole:SW_Hole_1u
- SW16, SW2, SW40, SW49, SW7 (x2): footprint kbd_SW_Hole:SW_Hole_1.25 -> kbd_SW_Hole:SW_Hole_1.25u
- SW5, SW6: footprint kbd_SW_Hole:SW_Hole_1.75 -> kbd_SW_Hole:SW_Hole_1.75u
