File: Keyboard/N51GL/2_Assemble/Naked51_Assemble.sch (KiCad schematic (older format))
At the start: 138 parts, among them J1 Conn_01x02, J10 Conn_01x01, J11 Conn_01x01, J12 Conn_01x01, J13 Conn_01x01, J14 Conn_01x01, J15 Conn_01x01, J16 Conn_01x01, J17 Conn_01x01, J2 Conn_01x01, J3 Conn_01x01, J4 Conn_01x01, J5 Conn_01x01, J6 Conn_01x01, J7 Conn_01x01, J8 Conn_01x01, J9 Conn_01x01, SW1 SW_PUSH, SW10 SW_PUSH, SW11 SW_PUSH, SW12 SW_PUSH, SW13 SW_PUSH, SW14 SW_PUSH, SW15 SW_PUSH, SW16 SW_PUSH, SW17 SW_PUSH, SW18 SW_PUSH, SW19 SW_PUSH, SW2 Rotary_Encoder_Switch, SW20 SW_PUSH, SW21 SW_PUSH, SW22 SW_PUSH, SW23 SW_PUSH, SW24 SW_PUSH, SW25 SW_PUSH, SW26 SW_PUSH, SW27 SW_PUSH, SW28 SW_PUSH, SW29 SW_PUSH, SW3 SW_PUSH, SW30 SW_PUSH, SW31 SW_PUSH, SW32 SW_PUSH, SW33 SW_PUSH, SW34 SW_PUSH, SW35 SW_PUSH, SW36 SW_PUSH, SW37 SW_PUSH, SW38 SW_PUSH, SW39 SW_PUSH, SW4 SW_PUSH, SW40 SW_PUSH, SW41 SW_PUSH, SW42 SW_PUSH, SW43 SW_PUSH, SW44 SW_PUSH, SW45 SW_PUSH, SW46 SW_PUSH, SW47 SW_PUSH, SW48 SW_PUSH, SW49 SW_PUSH, SW5 SW_PUSH, SW50 SW_PUSH, SW51 SW_PUSH, SW52 SW_PUSH, SW53 SW_PUSH, SW6 SW_PUSH, SW7 SW_PUSH, SW8 SW_PUSH, SW9 SW_PUSH, U1 BLEMicroPro

Commit message: バックアップファイルの整理
Parts:
- U1: symbol kbd:BLEMicroPro -> Salicylic_kbd:Micon_BLEMicroPro
Changed lines of the file:
@@
 BLE Micro Pro
 $Comp
-L kbd:BLEMicroPro U1
+L Salicylic_kbd:Micon_BLEMicroPro U1
 U 1 1 5BF16C54
 P 2150 1975

Commit message: シンボル、フットプリントの更新に合わせて更新
Parts:
- removed L10, L11, L12, L13, L14, L15, L2, L3, L4, L5, L6, L7, L8, L9: SK6812MINI, kbd_Parts:LED_SK6812MINI-E_BL, symbol kbd:SK6812MINI
- added L10, L11, L12, L13, L14, L15, L2, L3, L4, L5, L6, L7, L8, L9: SK6812MINI, kbd_Parts:LED_SK6812MINI-E_BL, symbol Salicylic_kbd:LED_SK6812MINI-E
- L1: symbol kbd:SK6812MINI -> Salicylic_kbd:LED_SK6812MINI-E
- SW1, SW10, SW11, SW12, SW13, SW14, SW15, SW16, SW17, SW18, SW19, SW20, SW21, SW22, SW23, SW24, SW25, SW26, SW27, SW28, SW29, SW3, SW30, SW31, SW32, SW33, SW34, SW35, SW36, SW37, SW38, SW39, SW4, SW40, SW41, SW42, SW43, SW44, SW45, SW46, SW47, SW48, SW49, SW5, SW50, SW51, SW52, SW53, SW6, SW7, SW8, SW9: symbol kbd:SW_PUSH -> Switch:SW_Push
Connections:
- wire segments 263 -> 159
Other:
- moved on the sheet: D1, D10, D11, D12, D13, D14, D15, D16, D17, D18, D19, D2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

Commit message: 使用するフットプリントを最新化
・EC12
・バッテリーピン
Parts:
- J1: footprint kbd_Parts:Battery_XH2.5_GL -> kbd_Parts:Battery_XH2.5_GL_PCB
- SW2: footprint kbd_Parts:RotaryEncoder_EC11E -> kbd_Parts:RotaryEncoder_EC12E
Changed lines of the file:
@@
 F 0 "J1" H 12443 1025 50  0000 C CNN
 F 1 "Conn_01x02" H 12443 1116 50  0000 C CNN
-F 2 "kbd_Parts:Battery_XH2.5_GL" H 12525 1350 50  0001 C CNN
+F 2 "kbd_Parts:Battery_XH2.5_GL_PCB" H 12525 1350 50  0001 C CNN
 F 3 "~" H 12525 1350 50  0001 C CNN
 	1    12525 1350
@@
 F 0 "SW2" V 2404 4955 50  0000 L CNN
 F 1 "Rotary_Encoder_Switch" V 2495 4955 50  0000 L CNN
-F 2 "kbd_Parts:RotaryEncoder_EC11E" H 2300 4885 50  0001 C CNN
+F 2 "kbd_Parts:RotaryEncoder_EC12E" H 2300 4885 50  0001 C CNN
 F 3 "~" H 2450 4985 50  0001 C CNN
 	1    2450 4725

Commit message: フットプリント名の変更に対応
Parts:
- SW1, SW11, SW12, SW13, SW14, SW15, SW16, SW18, SW19, SW20, SW22, SW23, SW24, SW25, SW26, SW27, SW28, SW29, SW3, SW30, SW31, SW32, SW34, SW35, SW36, SW38, SW39, SW40, SW41, SW42, SW43, SW44, SW46, SW47, SW48, SW50, SW51, SW52, SW7, SW8, SW9: footprint kbd_SW:CherryMX_Hotswap_1.0u -> kbd_SW:CherryMX_Hotswap_1u
- SW45, SW49: footprint kbd_SW:CherryMX_Hotswap_1.0u_Small1 -> kbd_SW:CherryMX_Hotswap_1u_Small1
